File: Hardware/days_worked_counter/days_worked_counter.kicad_sch (KiCad schematic)
At the start: 0 parts

Commit message: Add tidal force
Changed lines of the file:
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@@
     (stroke (width 0) (type default) (color 0 0 0 0))
+  )
+  (symbol (lib_id "KenwoodFox:TIDAL_FORCE_LOGO") (at 185.42 173.99 0) (unit 1)
+    (in_bom yes) (on_board yes) (fields_autoplaced)
+    (property "Reference" "#G101" (id 0) (at 185.42 167.0047 0)
+      (effects (font (size 1.27 1.27)) hide)
+    )
+    (property "Value" "TIDAL_FORCE_LOGO" (id 1) (at 185.42 180.9753 0)
+      (effects (font (size 1.27 1.27)) hide)
+    )
+    (property "Footprint" "KenwoodFox:TIDAL_FORCE_LOGO" (id 2) (at 185.42 173.99 0)
+      (effects (font (size 1.27 1.27)) hide)
+    )
+    (property "Datasheet" "" (id 3) (at 185.42 173.99 0)
+      (effects (font (size 1.27 1.27)) hide)
+    )
   )
   (sheet (at 127 86.36) (size 25.4 24.13) (fields_autoplaced)
@@
   )
   (symbol_instances
+    (path "/6c03b9a0-891c-4f2b-92c2-a6484d90febe"
+      (reference "#G101") (unit 1) (value "TIDAL_FORCE_LOGO") (footprint "KenwoodFox:TIDAL_FORCE_LOGO")
+    )
     (path "/5b3b94e9-8561-416b-92c8-c061c8d10891/7037ac14-17c8-466a-b4b8-2bf740656bda"
       (reference "#PWR0101") (unit 1) (value "+5V") (footprint "")

Commit message: Cleanup more stuff
Other:
- sheet Display Card renamed Display Card 0
- sheet Display Card1 renamed Display Card 1
- sheet Display Card2 renamed Display Card 2
- sheet MCU ports: added CLOCK_OUT, DATA_OUT, LATCH_OUT; removed none
Changed lines of the file:
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@@
   (no_connect (at 264.16 99.06))
   (no_connect (at 264.16 93.98))
+  (wire (pts (xy 152.4 99.06) (xy 162.56 99.06))
+    (stroke (width 0) (type default) (color 0 0 0 0))
+  )
   (wire (pts (xy 261.62 93.98) (xy 264.16 93.98))
     (stroke (width 0) (type default) (color 0 0 0 0))
@@
     (stroke (width 0) (type default) (color 0 0 0 0))
   )
+  (wire (pts (xy 152.4 93.98) (xy 162.56 93.98))
+    (stroke (width 0) (type default) (color 0 0 0 0))
+  )
   (wire (pts (xy 227.33 93.98) (xy 231.14 93.98))
     (stroke (width 0) (type default) (color 0 0 0 0))
   )
   (wire (pts (xy 261.62 99.06) (xy 264.16 99.06))
+    (stroke (width 0) (type default) (color 0 0 0 0))
+  )
+  (wire (pts (xy 152.4 96.52) (xy 162.56 96.52))
     (stroke (width 0) (type default) (color 0 0 0 0))
   )
@@
       (effects (font (size 1.27 1.27)) (justify left))
     )
+    (pin "DATA_OUT" output (at 152.4 93.98 0)
+      (effects (font (size 1.27 1.27)) (justify right))
+    )
+    (pin "CLOCK_OUT" output (at 152.4 96.52 0)
+      (effects (font (size 1.27 1.27)) (justify right))
+    )
+    (pin "LATCH_OUT" output (at 152.4 99.06 0)
+      (effects (font (size 1.27 1.27)) (justify right))
+    )
   )
   (sheet (at 93.98 86.36) (size 25.4 13.97) (fields_autoplaced)
@@
     (stroke (width 0.1524) (type solid) (color 0 0 0 0))
     (fill (color 0 0 0 0.0000))
-    (property "Sheet name" "Display Card2" (id 0) (at 231.14 90.7284 0)
+    (property "Sheet name" "Display Card 2" (id 0) (at 231.14 90.7284 0)
       (effects (font (size 1.27 1.27)) (justify left bottom))
     )
@@
     (stroke (width 0.1524) (type solid) (color 0 0 0 0))
     (fill (color 0 0 0 0.0000))
-    (property "Sheet name" "Display Card1" (id 0) (at 196.85 90.7284 0)
+    (property "Sheet name" "Display Card 1" (id 0) (at 196.85 90.7284 0)
       (effects (font (size 1.27 1.27)) (justify left bottom))
     )
@@
     (stroke (width 0.1524) (type solid) (color 0 0 0 0))
     (fill (color 0 0 0 0.0000))
-    (property "Sheet name" "Display Card" (id 0) (at 162.56 90.7284 0)
+    (property "Sheet name" "Display Card 0" (id 0) (at 162.56 90.7284 0)
       (effects (font (size 1.27 1.27)) (justify left bottom))
     )
@@
       (reference "#PWR0142") (unit 1) (value "GND") (footprint "")
     )
+    (path "/5b3b94e9-8561-416b-92c8-c061c8d10891/fcb60cea-8d01-4e21-9d42-e046c66cf084"
+      (reference "#PWR0143") (unit 1) (value "GND") (footprint "")
+    )
+    (path "/e578bf18-fecf-4fc4-8e6f-ece5d8a7ea5b/1bc305d3-036b-401d-a514-784eb0880730"
+      (reference "#PWR0144") (unit 1) (value "GND") (footprint "")
+    )
+    (path "/e578bf18-fecf-4fc4-8e6f-ece5d8a7ea5b/e44a2b3b-efc7-4a26-95e4-3c25f0f384da"
+      (reference "#PWR0145") (unit 1) (value "GND") (footprint "")
+    )
+    (path "/c6dca6b0-6120-4130-a5d8-8ac8450c22c0/1bc305d3-036b-401d-a514-784eb0880730"
+      (reference "#PWR0146") (unit 1) (value "GND") (footprint "")
+    )
+    (path "/c6dca6b0-6120-4130-a5d8-8ac8450c22c0/e44a2b3b-efc7-4a26-95e4-3c25f0f384da"
+      (reference "#PWR0147") (unit 1) (value "GND") (footprint "")
+    )
+    (path "/71dca6e4-949c-46c2-979f-90716fc3f3f2/1bc305d3-036b-401d-a514-784eb0880730"
+      (reference "#PWR0148") (unit 1) (value "GND") (footprint "")
+    )
+    (path "/71dca6e4-949c-46c2-979f-90716fc3f3f2/e44a2b3b-efc7-4a26-95e4-3c25f0f384da"
+      (reference "#PWR0149") (unit 1) (value "GND") (footprint "")
+    )
     (path "/5b3b94e9-8561-416b-92c8-c061c8d10891/d7b3bb76-b393-45be-9562-d4b1e8ae9a1b"
       (reference "C201") (unit 1) (value "4.7uf") (footprint "Capacitor_SMD:CP_Elec_4x3")
@@
       (reference "C701") (unit 1) (value "10uF") (footprint "Capacitor_SMD:C_0805_2012Metric")
     )
+    (path "/5b3b94e9-8561-416b-92c8-c061c8d10891/6e3d74ef-77f4-4bfd-8f5f-40b4652f917f"
+      (reference "D201") (unit 1) (value "STAT") (footprint "")
+    )
     (path "/6564c8a6-7134-401f-ba3c-a13a9f9d361c/f9529247-a826-47df-8b27-032fa786d97c"
       (reference "D301") (unit 1) (value "RX") (footprint "LED_SMD:LED_0805_2012Metric")
@@
       (reference "J401") (unit 1) (value "19V Input") (footprint "Connector_BarrelJack:BarrelJack_GCT_DCJ200-10-A_Horizontal")
     )
+    (path "/e578bf18-fecf-4fc4-8e6f-ece5d8a7ea5b/0e0f3db3-64f0-4ff6-b5d0-f6b4e3826e0a"
+      (reference "Q501") (unit 1) (value "MMBT3904") (footprint "Package_TO_SOT_SMD:SOT-23")
+    )
+    (path "/c6dca6b0-6120-4130-a5d8-8ac8450c22c0/0e0f3db3-64f0-4ff6-b5d0-f6b4e3826e0a"
+      (reference "Q601") (unit 1) (value "MMBT3904") (footprint "Package_TO_SOT_SMD:SOT-23")
+    )
+    (path "/71dca6e4-949c-46c2-979f-90716fc3f3f2/0e0f3db3-64f0-4ff6-b5d0-f6b4e3826e0a"
+      (reference "Q701") (unit 1) (value "MMBT3904") (footprint "Package_TO_SOT_SMD:SOT-23")
+    )
     (path "/5b3b94e9-8561-416b-92c8-c061c8d10891/70d215ad-7fe4-43ad-9cda-3f9fe39c67d6"
       (reference "R201") (unit 1) (value "1K") (footprint "Resistor_SMD:R_0805_2012Metric")
@@
       (reference "R203") (unit 1) (value "1K") (footprint "Resistor_SMD:R_0805_2012Metric")
     )
+    (path "/5b3b94e9-8561-416b-92c8-c061c8d10891/9b3f3b36-c8e8-40fb-bfd8-3faa6dde2f59"
+      (reference "R204") (unit 1) (value "1K") (footprint "Resistor_SMD:R_0805_2012Metric")
+    )
     (path "/6564c8a6-7134-401f-ba3c-a13a9f9d361c/9aac1638-86a7-4ebe-8c13-efdabdb19e93"
       (reference "R301") (unit 1) (value "1K") (footprint "Resistor_SMD:R_0805_2012Metric")
@@
       (reference "R401") (unit 1) (value "1K") (footprint "Resistor_SMD:R_0805_2012Metric")
     )
+    (path "/e578bf18-fecf-4fc4-8e6f-ece5d8a7ea5b/b09c2764-8d02-4f54-b781-9c6aad282eaf"
+      (reference "R501") (unit 1) (value "10K") (footprint "Resistor_SMD:R_0805_2012Metric")
+    )
+    (path "/c6dca6b0-6120-4130-a5d8-8ac8450c22c0/b09c2764-8d02-4f54-b781-9c6aad282eaf"
+      (reference "R601") (unit 1) (value "10K") (footprint "Resistor_SMD:R_0805_2012Metric")
+    )
+    (path "/71dca6e4-949c-46c2-979f-90716fc3f3f2/b09c2764-8d02-4f54-b781-9c6aad282eaf"
+      (reference "R701") (unit 1) (value "10K") (footprint "Resistor_SMD:R_0805_2012Metric")
+    )
+    (path "/c6dca6b0-6120-4130-a5d8-8ac8450c22c0/a633266d-1627-4e1b-ac68-73eadcc4dfa6"
+      (reference "R?") (unit 1) (value "750R?") (footprint "Resistor_SMD:R_0805_2012Metric")
+    )
+    (path "/71dca6e4-949c-46c2-979f-90716fc3f3f2/a633266d-1627-4e1b-ac68-73eadcc4dfa6"
+      (reference "R?") (unit 1) (value "750R?") (footprint "Resistor_SMD:R_0805_2012Metric")
+    )
+    (path "/e578bf18-fecf-4fc4-8e6f-ece5d8a7ea5b/a633266d-1627-4e1b-ac68-73eadcc4dfa6"
+      (reference "R?") (unit 1) (value "750R?") (footprint "Resistor_SMD:R_0805_2012Metric")
+    )
     (path "/5b3b94e9-8561-416b-92c8-c061c8d10891/a7079559-26b6-43bc-86a7-dfee96e5ef94"

Commit message: Add all the cool stuff
Other:
- company: (none) -> FRC 1721
- title: (none) -> Days Without Incident Sign

Commit message: get input from @ka2qfx
Parts:
- added J101, J103, J105: OUT, Connector_PinSocket_2.54mm:PinSocket_1x06_P2.54mm_Vertical, symbol Connector_Generic:Conn_01x06
- added J102, J104: IN, Connector_PinSocket_2.54mm:PinSocket_1x06_P2.54mm_Vertical, symbol Connector_Generic:Conn_01x06
Connections:
- net Display Card 0/CLOCK_OUT: now also J101.3 (Pin_3)
- net Display Card 0/DATA_OUT: now also J101.2 (Pin_2)
- net Display Card 0/LATCH_OUT: now also J101.4 (Pin_4)
- net Display Card 1/CLOCK_OUT: now also J103.3 (Pin_3)
- net Display Card 1/DATA_OUT: now also J103.2 (Pin_2)
- net Display Card 1/LATCH_OUT: now also J103.4 (Pin_4)
- net Display Card 2/CLOCK_OUT: now also J105.3 (Pin_3)
- net Display Card 2/DATA_OUT: now also J105.2 (Pin_2)
- net Display Card 2/LATCH_OUT: now also J105.4 (Pin_4)
- new net +19V: J101.1 (Pin_1), J102.1 (Pin_1), J103.1 (Pin_1), J104.1 (Pin_1), J105.1 (Pin_1)
- new net +5V: J101.5 (Pin_5), J102.5 (Pin_5), J103.5 (Pin_5), J104.5 (Pin_5), J105.5 (Pin_5)
- new net Display Card 1/CLOCK_IN: J102.3 (Pin_3)
- new net Display Card 1/DATA_IN: J102.2 (Pin_2)
- new net Display Card 1/LATCH_IN: J102.4 (Pin_4)
- new net Display Card 2/CLOCK_IN: J104.3 (Pin_3)
- new net Display Card 2/DATA_IN: J104.2 (Pin_2)
- new net Display Card 2/LATCH_IN: J104.4 (Pin_4)
- new net GND: J101.6 (Pin_6), J102.6 (Pin_6), J103.6 (Pin_6), J104.6 (Pin_6), J105.6 (Pin_6)
- no-connect marks 3 -> 0
