File: Hardware/days_worked_counter/display_card.kicad_sch (KiCad schematic)
At the start: 4 parts, among them J501 Top Conn, J502 Bottom Conn, U501 SN74HC595

Commit message: With thanks to @ka2qfx
Parts:
- renumbered J502 to J501, J501 to J502
Changed lines of the file:
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@@
   (symbol (lib_id "Connector_Generic:Conn_01x09") (at 34.29 74.295 90) (unit 1)
     (in_bom yes) (on_board yes)
-    (property "Reference" "J501" (id 0) (at 27.305 71.755 90)
+    (property "Reference" "J502" (id 0) (at 27.305 71.755 90)
       (effects (font (size 1.27 1.27)) (justify left))
     )
@@
   (symbol (lib_id "power:GND") (at 102.87 116.205 0) (unit 1)
     (in_bom yes) (on_board yes)
-    (property "Reference" "#PWR0126" (id 0) (at 102.87 122.555 0)
+    (property "Reference" "#PWR0508" (id 0) (at 102.87 122.555 0)
       (effects (font (size 1.27 1.27)) hide)
     )
@@
   (symbol (lib_id "power:GND") (at 88.9 83.185 0) (unit 1)
     (in_bom yes) (on_board yes)
-    (property "Reference" "#PWR0130" (id 0) (at 88.9 89.535 0)
+    (property "Reference" "#PWR0506" (id 0) (at 88.9 89.535 0)
       (effects (font (size 1.27 1.27)) hide)
     )
@@
   (symbol (lib_id "power:+5V") (at 71.12 102.235 0) (unit 1)
     (in_bom yes) (on_board yes)
-    (property "Reference" "#PWR0127" (id 0) (at 71.12 106.045 0)
+    (property "Reference" "#PWR0503" (id 0) (at 71.12 106.045 0)
       (effects (font (size 1.27 1.27)) hide)
     )
@@
   (symbol (lib_id "power:GND") (at 74.93 97.155 0) (unit 1)
     (in_bom yes) (on_board yes)
-    (property "Reference" "#PWR0128" (id 0) (at 74.93 103.505 0)
+    (property "Reference" "#PWR0504" (id 0) (at 74.93 103.505 0)
       (effects (font (size 1.27 1.27)) hide)
     )
@@
   (symbol (lib_id "power:+5V") (at 102.87 84.455 0) (unit 1)
     (in_bom yes) (on_board yes)
-    (property "Reference" "#PWR0125" (id 0) (at 102.87 88.265 0)
+    (property "Reference" "#PWR0507" (id 0) (at 102.87 88.265 0)
       (effects (font (size 1.27 1.27)) hide)
     )
@@
   (symbol (lib_id "Connector_Generic:Conn_01x09") (at 33.02 121.285 90) (mirror x) (unit 1)
     (in_bom yes) (on_board yes)
-    (property "Reference" "J502" (id 0) (at 45.085 123.825 90)
+    (property "Reference" "J501" (id 0) (at 45.085 123.825 90)
       (effects (font (size 1.27 1.27)) (justify left))
     )
@@
   (symbol (lib_id "power:+5V") (at 88.9 75.565 0) (unit 1)
     (in_bom yes) (on_board yes)
-    (property "Reference" "#PWR0129" (id 0) (at 88.9 79.375 0)
+    (property "Reference" "#PWR0505" (id 0) (at 88.9 79.375 0)
       (effects (font (size 1.27 1.27)) hide)
     )
@@
   (symbol (lib_id "power:GND") (at 34.29 82.55 0) (unit 1)
     (in_bom yes) (on_board yes)
-    (property "Reference" "#PWR0222" (id 0) (at 34.29 88.9 0)
+    (property "Reference" "#PWR0501" (id 0) (at 34.29 88.9 0)
       (effects (font (size 1.27 1.27)) hide)
     )
@@
   (symbol (lib_id "power:GND") (at 49.53 116.84 0) (unit 1)
     (in_bom yes) (on_board yes)
-    (property "Reference" "#PWR0166" (id 0) (at 49.53 123.19 0)
+    (property "Reference" "#PWR0502" (id 0) (at 49.53 123.19 0)
       (effects (font (size 1.27 1.27)) hide)
     )
