File: Hardware/days_worked_counter/Power.kicad_sch (KiCad schematic)
At the start: 5 parts, among them J401 19V Input, U401 LM1117-5.0

Commit message: Add all the cool stuff
Other:
- company: (none) -> FRC 1721
- title: (none) -> Days Without Incident Sign
Changed lines of the file:
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@@
 (kicad_sch (version 20211123) (generator eeschema)
   (paper "A4")
+  (title_block
+    (title "Days Without Incident Sign")
+    (date "2022-06-24")
+    (rev "v0.1-RC1")
+    (company "FRC 1721")
+  )
   (junction (at 160.02 88.9) (diameter 0) (color 0 0 0 0)
   )

Commit message: Even more stuff
Changed lines of the file:
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@@
   (symbol (lib_id "Connector:Barrel_Jack") (at 125.73 91.44 0) (unit 1)
     (in_bom yes) (on_board yes)
-    (property "Reference" "J401" (id 0) (at 125.73 82.55 0))
+    (property "Reference" "J401" (id 0) (at 125.73 84.455 0))
     (property "Value" "19V Input" (id 1) (at 125.73 86.36 0))
     (property "Footprint" "Connector_BarrelJack:BarrelJack_GCT_DCJ200-10-A_Horizontal" (id 2) (at 127 92.456 0)

Commit message: Add stuff
Connections:
- net +19V: now reaches J401.1, U401.3 (VI)
Changed lines of the file:
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@@
   (junction (at 160.02 88.9) (diameter 0) (color 0 0 0 0)
+  )
+  (junction (at 137.16 88.9) (diameter 0) (color 0 0 0 0)
   )
   (junction (at 158.75 88.9) (diameter 0) (color 0 0 0 0)
   )
   (wire (pts (xy 137.16 93.98) (xy 133.35 93.98))
+    (stroke (width 0) (type default) (color 0 0 0 0))
+  )
+  (wire (pts (xy 137.16 86.36) (xy 137.16 88.9))
     (stroke (width 0) (type default) (color 0 0 0 0))
   )
@@
     (stroke (width 0) (type default) (color 0 0 0 0))
   )
-  (wire (pts (xy 133.35 88.9) (xy 140.97 88.9))
+  (wire (pts (xy 133.35 88.9) (xy 137.16 88.9))
     (stroke (width 0) (type default) (color 0 0 0 0))
   )
@@
     (stroke (width 0) (type default) (color 0 0 0 0))
   )
+  (wire (pts (xy 137.16 88.9) (xy 140.97 88.9))
+    (stroke (width 0) (type default) (color 0 0 0 0))
+  )
   (text "I dont think this regulator can\ntake this\nvoltage, ask Mark."
-    (at 128.27 82.55 0)
+    (at 113.03 79.375 0)
     (effects (font (size 1.27 1.27)) (justify left bottom))
   )
@@
     )
     (property "Datasheet" "" (id 3) (at 160.02 97.79 0)
+      (effects (font (size 1.27 1.27)) hide)
+    )
+    (pin "1")
+  )
+  (symbol (lib_id "KenwoodFox:+19V") (at 137.16 86.36 0) (unit 1)
+    (in_bom yes) (on_board yes)
+    (property "Reference" "#PWR?" (id 0) (at 137.16 90.17 0)
+      (effects (font (size 1.27 1.27)) hide)
+    )
+    (property "Value" "+19V" (id 1) (at 137.16 82.55 0))
+    (property "Footprint" "" (id 2) (at 137.16 86.36 0)
+      (effects (font (size 1.27 1.27)) hide)
+    )
+    (property "Datasheet" "" (id 3) (at 137.16 86.36 0)
       (effects (font (size 1.27 1.27)) hide)
     )
@@
   (symbol (lib_id "Device:C_Small") (at 160.02 93.98 0) (unit 1)
     (in_bom yes) (on_board yes)
-    (property "Reference" "C401" (id 0) (at 163.83 93.98 0))
+    (property "Reference" "C401" (id 0) (at 164.465 94.615 0))
     (property "Value" "100nF" (id 1) (at 165.1 96.52 0))
     (property "Footprint" "Capacitor_SMD:C_0805_2012Metric" (id 2) (at 160.02 93.98 0)
