File: Hardware/days_worked_counter/buffer.kicad_sch (KiCad schematic)
At the start: 5 parts, among them Q801 MMBT3904, Q802 MMBT3906

Commit message: With thanks to @ka2qfx
Parts:
- renumbered Q801 to Q601, Q802 to Q602, R801 to R601, R802 to R602, R803 to R603
Changed lines of the file:
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@@
   (symbol (lib_id "Device:R_Small") (at 139.065 99.06 90) (unit 1)
     (in_bom yes) (on_board yes)
-    (property "Reference" "R801" (id 0) (at 138.43 100.965 90))
+    (property "Reference" "R601" (id 0) (at 138.43 100.965 90))
     (property "Value" "10K" (id 1) (at 139.065 102.87 90))
     (property "Footprint" "Resistor_SMD:R_0805_2012Metric" (id 2) (at 139.065 99.06 0)
@@
   (symbol (lib_id "power:GND") (at 150.495 106.68 0) (unit 1)
     (in_bom yes) (on_board yes)
-    (property "Reference" "#PWR0145" (id 0) (at 150.495 113.03 0)
+    (property "Reference" "#PWR0601" (id 0) (at 150.495 113.03 0)
       (effects (font (size 1.27 1.27)) hide)
     )
@@
   (symbol (lib_id "KenwoodFox:+19V") (at 166.37 85.725 0) (unit 1)
     (in_bom yes) (on_board yes)
-    (property "Reference" "#PWR0144" (id 0) (at 166.37 89.535 0)
+    (property "Reference" "#PWR0602" (id 0) (at 166.37 89.535 0)
       (effects (font (size 1.27 1.27)) hide)
     )
@@
   (symbol (lib_id "Device:R_Small") (at 170.815 99.06 90) (unit 1)
     (in_bom yes) (on_board yes)
-    (property "Reference" "R803" (id 0) (at 167.64 100.965 90))
+    (property "Reference" "R603" (id 0) (at 167.64 100.965 90))
     (property "Value" "250R" (id 1) (at 168.91 102.87 90))
     (property "Footprint" "Resistor_SMD:R_0805_2012Metric" (id 2) (at 170.815 99.06 0)
@@
   (symbol (lib_id "Device:R_Small") (at 154.94 92.075 90) (unit 1)
     (in_bom yes) (on_board yes)
-    (property "Reference" "R802" (id 0) (at 154.305 87.63 90))
+    (property "Reference" "R602" (id 0) (at 154.305 87.63 90))
     (property "Value" "2K2" (id 1) (at 154.94 89.535 90))
     (property "Footprint" "Resistor_SMD:R_0805_2012Metric" (id 2) (at 154.94 92.075 0)
@@
   (symbol (lib_id "Transistor_BJT:MMBT3906") (at 163.83 92.075 0) (mirror x) (unit 1)
     (in_bom yes) (on_board yes)
-    (property "Reference" "Q802" (id 0) (at 168.91 90.805 0)
+    (property "Reference" "Q602" (id 0) (at 168.91 90.805 0)
       (effects (font (size 1.27 1.27)) (justify left))
     )
@@
   (symbol (lib_id "Transistor_BJT:MMBT3904") (at 147.955 99.06 0) (unit 1)
     (in_bom yes) (on_board yes) (fields_autoplaced)
-    (property "Reference" "Q801" (id 0) (at 153.035 97.7899 0)
+    (property "Reference" "Q601" (id 0) (at 153.035 97.7899 0)
       (effects (font (size 1.27 1.27)) (justify left))
     )
