File: Hardware/days_worked_counter/days_worked_counter.kicad_pcb (KiCad board)
At the start: 2 copper layers, 114.5 x 141 mm, 69 parts, among them J101 OUT, J102 IN, J103 OUT, J104 IN, J105 OUT, J301 USB_B_Micro, J302 PROG, J401 19V Input, J501 Top Conn, J502 Bottom Conn, J601 Top Conn, J602 Bottom Conn, J701 Top Conn, J702 Bottom Conn, Q501 MMBT3904, Q601 MMBT3904, Q701 MMBT3904, SW201 RESET, SW202 DAY_RESET, SW203 DAY_ADV, SW204 DAY_SUB, U201 ATmega328P-A, U202 DS1307Z+, U301 FT232RL, U401 LM1117-5.0, U501 SN74HC595, U601 SN74HC595, U701 SN74HC595, Y201 16mHz, Y202 32.768kHz

Commit message: Thank @ka2qfx for fixups!
Parts:
- added Q501: MMBT3904, Package_TO_SOT_SMD:SOT-23, F.Cu at (108.2, -87.5)
- added Q502: MMBT3904, Package_TO_SOT_SMD:SOT-23, F.Cu at (98.5, -87.5)
- added Q503: MMBT3904, Package_TO_SOT_SMD:SOT-23, F.Cu at (118.0, -87.5)
- added Q504: MMBT3904, Package_TO_SOT_SMD:SOT-23, F.Cu at (108.2, -83.0)
- added Q505: MMBT3906, Package_TO_SOT_SMD:SOT-23, F.Cu at (103.4, -87.5)
- added Q506: MMBT3906, Package_TO_SOT_SMD:SOT-23, F.Cu at (98.5, -83.0)
- added Q507: MMBT3906, Package_TO_SOT_SMD:SOT-23, F.Cu at (113.1, -83.0)
- added Q508: MMBT3904, Package_TO_SOT_SMD:SOT-23, F.Cu at (103.4, -78.6)
- added Q509: MMBT3906, Package_TO_SOT_SMD:SOT-23, F.Cu at (103.4, -74.2)
- added Q510: MMBT3904, Package_TO_SOT_SMD:SOT-23, F.Cu at (113.1, -87.5)
- added Q511: MMBT3904, Package_TO_SOT_SMD:SOT-23, F.Cu at (103.4, -83.0)
- added Q513: MMBT3906, Package_TO_SOT_SMD:SOT-23, F.Cu at (98.5, -78.6)
- added Q514: MMBT3906, Package_TO_SOT_SMD:SOT-23, F.Cu at (108.2, -78.6)
- added Q515: MMBT3906, Package_TO_SOT_SMD:SOT-23, F.Cu at (98.5, -74.2)
- added Q601: MMBT3904, Package_TO_SOT_SMD:SOT-23, F.Cu at (66.8, -62.9)
- added Q602: MMBT3904, Package_TO_SOT_SMD:SOT-23, F.Cu at (57.0, -62.9)
- added Q603: MMBT3904, Package_TO_SOT_SMD:SOT-23, F.Cu at (76.6, -62.9)
- added Q604: MMBT3904, Package_TO_SOT_SMD:SOT-23, F.Cu at (66.8, -58.4)
- added Q605: MMBT3906, Package_TO_SOT_SMD:SOT-23, F.Cu at (61.9, -62.9)
- added Q606: MMBT3906, Package_TO_SOT_SMD:SOT-23, F.Cu at (57.0, -58.4)
- added Q607: MMBT3906, Package_TO_SOT_SMD:SOT-23, F.Cu at (71.7, -58.4)
- added Q608: MMBT3904, Package_TO_SOT_SMD:SOT-23, F.Cu at (61.9, -54.0)
- added Q609: MMBT3906, Package_TO_SOT_SMD:SOT-23, F.Cu at (61.9, -49.5)
- added Q610: MMBT3904, Package_TO_SOT_SMD:SOT-23, F.Cu at (71.7, -62.9)
- added Q611: MMBT3904, Package_TO_SOT_SMD:SOT-23, F.Cu at (61.9, -58.4)
- added Q613: MMBT3906, Package_TO_SOT_SMD:SOT-23, F.Cu at (57.0, -54.0)
- added Q614: MMBT3906, Package_TO_SOT_SMD:SOT-23, F.Cu at (66.8, -54.0)
- added Q615: MMBT3906, Package_TO_SOT_SMD:SOT-23, F.Cu at (57.0, -49.5)
- added Q701: MMBT3904, Package_TO_SOT_SMD:SOT-23, F.Cu at (66.8, -87.5)
- added Q702: MMBT3904, Package_TO_SOT_SMD:SOT-23, F.Cu at (57.0, -87.5)
- added Q703: MMBT3904, Package_TO_SOT_SMD:SOT-23, F.Cu at (76.6, -87.5)
- added Q704: MMBT3904, Package_TO_SOT_SMD:SOT-23, F.Cu at (66.8, -83.0)
- added Q705: MMBT3906, Package_TO_SOT_SMD:SOT-23, F.Cu at (61.9, -87.5)
- added Q706: MMBT3906, Package_TO_SOT_SMD:SOT-23, F.Cu at (57.0, -83.0)
- added Q707: MMBT3906, Package_TO_SOT_SMD:SOT-23, F.Cu at (71.7, -83.0)
- added Q708: MMBT3904, Package_TO_SOT_SMD:SOT-23, F.Cu at (61.9, -78.6)
- added Q709: MMBT3906, Package_TO_SOT_SMD:SOT-23, F.Cu at (61.9, -74.2)
- added Q710: MMBT3904, Package_TO_SOT_SMD:SOT-23, F.Cu at (71.7, -87.5)
- added Q711: MMBT3904, Package_TO_SOT_SMD:SOT-23, F.Cu at (61.9, -83.0)
- added Q713: MMBT3906, Package_TO_SOT_SMD:SOT-23, F.Cu at (57.0, -78.6)
- added Q714: MMBT3906, Package_TO_SOT_SMD:SOT-23, F.Cu at (66.8, -78.6)
- added Q715: MMBT3906, Package_TO_SOT_SMD:SOT-23, F.Cu at (57.0, -74.2)
- added R501: 10K, Resistor_SMD:R_0805_2012Metric, F.Cu at (107.0, -70.5)
- added R502: 10K, Resistor_SMD:R_0805_2012Metric, F.Cu at (108.0, -74.9)
- added R503: 10K, Resistor_SMD:R_0805_2012Metric, F.Cu at (122.7, -85.3)
- added R504: 10K, Resistor_SMD:R_0805_2012Metric, F.Cu at (112.9, -79.3)
- added R505: 2K2, Resistor_SMD:R_0805_2012Metric, F.Cu at (112.4, -73.5)
- added R506: 2K2, Resistor_SMD:R_0805_2012Metric, F.Cu at (111.5, -70.5)
- added R507: 2K2, Resistor_SMD:R_0805_2012Metric, F.Cu at (122.7, -88.2)
- added R508: 2K2, Resistor_SMD:R_0805_2012Metric, F.Cu at (127.1, -88.2)
- added R509: 250R, Resistor_SMD:R_0805_2012Metric, F.Cu at (117.3, -75.0)
- added R510: 250R, Resistor_SMD:R_0805_2012Metric, F.Cu at (122.2, -82.3)
- added R511: 250R, Resistor_SMD:R_0805_2012Metric, F.Cu at (117.8, -80.8)
- added R512: 10K, Resistor_SMD:R_0805_2012Metric, F.Cu at (112.9, -76.4)
- added R513: 10K, Resistor_SMD:R_0805_2012Metric, F.Cu at (122.2, -79.4)
- added R514: 10K, Resistor_SMD:R_0805_2012Metric, F.Cu at (102.6, -70.5)
- added R516: 2K2, Resistor_SMD:R_0805_2012Metric, F.Cu at (98.2, -70.5)
- added R517: 250R, Resistor_SMD:R_0805_2012Metric, F.Cu at (115.9, -70.5)
- added R518: 2K2, Resistor_SMD:R_0805_2012Metric, F.Cu at (117.8, -83.8)
- added R519: 2K2, Resistor_SMD:R_0805_2012Metric, F.Cu at (127.1, -85.3)
- added R521: 250R, Resistor_SMD:R_0805_2012Metric, F.Cu at (131.5, -88.2)
- added R522: 250R, Resistor_SMD:R_0805_2012Metric, F.Cu at (126.6, -82.3)
- added R523: 250R, Resistor_SMD:R_0805_2012Metric, F.Cu at (117.3, -77.9)
- added R601: 10K, Resistor_SMD:R_0805_2012Metric, F.Cu at (65.6, -45.8)
- added R602: 10K, Resistor_SMD:R_0805_2012Metric, F.Cu at (66.5, -50.3)
- added R603: 10K, Resistor_SMD:R_0805_2012Metric, F.Cu at (81.2, -60.7)
- added R604: 10K, Resistor_SMD:R_0805_2012Metric, F.Cu at (71.4, -54.7)
- added R605: 2K2, Resistor_SMD:R_0805_2012Metric, F.Cu at (71.0, -48.8)
- added R606: 2K2, Resistor_SMD:R_0805_2012Metric, F.Cu at (70.0, -45.9)
- added R607: 2K2, Resistor_SMD:R_0805_2012Metric, F.Cu at (81.2, -63.6)
- added R608: 2K2, Resistor_SMD:R_0805_2012Metric, F.Cu at (85.6, -63.6)
- added R609: 250R, Resistor_SMD:R_0805_2012Metric, F.Cu at (75.8, -50.3)
- added R610: 250R, Resistor_SMD:R_0805_2012Metric, F.Cu at (80.7, -57.7)
- added R611: 250R, Resistor_SMD:R_0805_2012Metric, F.Cu at (76.3, -56.2)
- added R612: 10K, Resistor_SMD:R_0805_2012Metric, F.Cu at (71.4, -51.8)
- added R613: 10K, Resistor_SMD:R_0805_2012Metric, F.Cu at (80.7, -54.8)
- added R614: 10K, Resistor_SMD:R_0805_2012Metric, F.Cu at (61.2, -45.8)
- added R616: 2K2, Resistor_SMD:R_0805_2012Metric, F.Cu at (56.8, -45.8)
- added R617: 250R, Resistor_SMD:R_0805_2012Metric, F.Cu at (74.4, -45.9)
- added R618: 2K2, Resistor_SMD:R_0805_2012Metric, F.Cu at (76.3, -59.2)
- added R619: 2K2, Resistor_SMD:R_0805_2012Metric, F.Cu at (85.6, -60.7)
- added R621: 250R, Resistor_SMD:R_0805_2012Metric, F.Cu at (90.0, -63.6)
- added R622: 250R, Resistor_SMD:R_0805_2012Metric, F.Cu at (85.2, -57.7)
- added R623: 250R, Resistor_SMD:R_0805_2012Metric, F.Cu at (75.8, -53.3)
- added R701: 10K, Resistor_SMD:R_0805_2012Metric, F.Cu at (65.6, -70.5)
- added R702: 10K, Resistor_SMD:R_0805_2012Metric, F.Cu at (66.5, -74.9)
- added R703: 10K, Resistor_SMD:R_0805_2012Metric, F.Cu at (81.2, -85.3)
- added R704: 10K, Resistor_SMD:R_0805_2012Metric, F.Cu at (71.4, -79.3)
- added R705: 2K2, Resistor_SMD:R_0805_2012Metric, F.Cu at (71.0, -73.5)
- added R706: 2K2, Resistor_SMD:R_0805_2012Metric, F.Cu at (70.0, -70.5)
- added R707: 2K2, Resistor_SMD:R_0805_2012Metric, F.Cu at (81.2, -88.2)
- added R708: 2K2, Resistor_SMD:R_0805_2012Metric, F.Cu at (85.6, -88.2)
- added R709: 250R, Resistor_SMD:R_0805_2012Metric, F.Cu at (75.8, -75.0)
- added R710: 250R, Resistor_SMD:R_0805_2012Metric, F.Cu at (80.7, -82.3)
- added R711: 250R, Resistor_SMD:R_0805_2012Metric, F.Cu at (76.3, -80.8)
- added R712: 10K, Resistor_SMD:R_0805_2012Metric, F.Cu at (71.4, -76.4)
- added R713: 10K, Resistor_SMD:R_0805_2012Metric, F.Cu at (80.7, -79.4)
- added R714: 10K, Resistor_SMD:R_0805_2012Metric, F.Cu at (61.2, -70.5)
- added R716: 2K2, Resistor_SMD:R_0805_2012Metric, F.Cu at (56.8, -70.5)
- added R717: 250R, Resistor_SMD:R_0805_2012Metric, F.Cu at (74.4, -70.5)
- added R718: 2K2, Resistor_SMD:R_0805_2012Metric, F.Cu at (76.3, -83.8)
- added R719: 2K2, Resistor_SMD:R_0805_2012Metric, F.Cu at (85.6, -85.3)
- added R721: 250R, Resistor_SMD:R_0805_2012Metric, F.Cu at (90.0, -88.2)
- added R722: 250R, Resistor_SMD:R_0805_2012Metric, F.Cu at (85.2, -82.3)
- added R723: 250R, Resistor_SMD:R_0805_2012Metric, F.Cu at (75.8, -77.9)
Connections:
- J501 pad 5: unconnected-(J501-Pad5) -> GND
- J502 pad 1: /Display Card 0/SEG_H_LAMP -> unconnected-(J502-Pad1)
- J601 pad 5: unconnected-(J601-Pad5) -> GND
- J602 pad 1: /Display Card 1/SEG_H_LAMP -> unconnected-(J602-Pad1)
- J701 pad 5: unconnected-(J701-Pad5) -> GND
- J702 pad 1: /Display Card 2/SEG_H_LAMP -> unconnected-(J702-Pad1)
- U501 pad 7: /Display Card 0/SEG_H -> unconnected-(U501-Pad7)
- U601 pad 7: /Display Card 1/SEG_H -> unconnected-(U601-Pad7)
- U701 pad 7: /Display Card 2/SEG_H -> unconnected-(U701-Pad7)

Commit message: Change direction
Parts:
- removed the Q501 at (108.2, -87.5)
- removed Q502, Q503, Q504, Q508, Q510, Q511, Q602, Q603, Q604, Q608, Q610, Q611, Q702, Q703, Q704, Q708, Q710, Q711: MMBT3904, Package_TO_SOT_SMD:SOT-23
- removed Q505, Q506, Q507, Q509, Q513, Q514, Q515, Q605, Q606, Q607, Q609, Q613, Q614, Q615, Q705, Q706, Q707, Q709, Q713, Q714, Q715: MMBT3906, Package_TO_SOT_SMD:SOT-23
- removed the Q601 at (66.8, -62.9)
- removed the Q701 at (66.8, -87.5)
- removed the R501 at (107.0, -70.5)
- removed R502, R503, R504, R512, R513, R514, R602, R603, R604, R612, R613, R614, R702, R703, R704, R712, R713, R714: 10K, Resistor_SMD:R_0805_2012Metric
- removed R505, R506, R507, R508, R516, R518, R519, R605, R606, R607, R608, R616, R618, R619, R705, R706, R707, R708, R716, R718, R719: 2K2, Resistor_SMD:R_0805_2012Metric
- removed R509, R510, R511, R517, R521, R522, R523, R609, R610, R611, R617, R621, R622, R623, R709, R710, R711, R717, R721, R722, R723: 250R, Resistor_SMD:R_0805_2012Metric
- removed the R601 at (65.6, -45.8)
- removed the R701 at (65.6, -70.5)
- added Q1001: MMBT3904, Package_TO_SOT_SMD:SOT-23, F.Cu at (85.0, -50.8)
- added Q1002: MMBT3906, Package_TO_SOT_SMD:SOT-23, F.Cu at (80.1, -50.8)
- added Q1101: MMBT3904, Package_TO_SOT_SMD:SOT-23, F.Cu at (85.0, -73.2)
- added Q1102: MMBT3906, Package_TO_SOT_SMD:SOT-23, F.Cu at (80.1, -73.2)
- added Q1201: MMBT3904, Package_TO_SOT_SMD:SOT-23, F.Cu at (67.5, -84.3)
- added Q1202: MMBT3906, Package_TO_SOT_SMD:SOT-23, F.Cu at (62.6, -84.3)
- added Q1301: MMBT3904, Package_TO_SOT_SMD:SOT-23, F.Cu at (137.6, -73.2)
- added Q1302: MMBT3906, Package_TO_SOT_SMD:SOT-23, F.Cu at (132.7, -73.2)
- added Q1401: MMBT3904, Package_TO_SOT_SMD:SOT-23, F.Cu at (67.5, -73.2)
- added Q1402: MMBT3906, Package_TO_SOT_SMD:SOT-23, F.Cu at (62.6, -73.2)
- added Q1501: MMBT3904, Package_TO_SOT_SMD:SOT-23, F.Cu at (67.5, -62.0)
- added Q1502: MMBT3906, Package_TO_SOT_SMD:SOT-23, F.Cu at (62.6, -62.0)
- added Q1601: MMBT3904, Package_TO_SOT_SMD:SOT-23, F.Cu at (102.5, -73.2)
- added Q1602: MMBT3906, Package_TO_SOT_SMD:SOT-23, F.Cu at (97.6, -73.2)
- added Q1701: MMBT3904, Package_TO_SOT_SMD:SOT-23, F.Cu at (120.1, -84.3)
- added Q1702: MMBT3906, Package_TO_SOT_SMD:SOT-23, F.Cu at (115.2, -84.3)
- added Q1801: MMBT3904, Package_TO_SOT_SMD:SOT-23, F.Cu at (137.6, -84.3)
- added Q1802: MMBT3906, Package_TO_SOT_SMD:SOT-23, F.Cu at (132.7, -84.3)
- added Q1901: MMBT3904, Package_TO_SOT_SMD:SOT-23, F.Cu at (120.1, -62.0)
- added Q1902: MMBT3906, Package_TO_SOT_SMD:SOT-23, F.Cu at (115.2, -62.0)
- added Q2001: MMBT3904, Package_TO_SOT_SMD:SOT-23, F.Cu at (102.5, -84.3)
- added Q2002: MMBT3906, Package_TO_SOT_SMD:SOT-23, F.Cu at (97.6, -84.3)
- added Q2101: MMBT3904, Package_TO_SOT_SMD:SOT-23, F.Cu at (67.5, -50.8)
- added Q2102: MMBT3906, Package_TO_SOT_SMD:SOT-23, F.Cu at (62.6, -50.8)
- added Q2201: MMBT3904, Package_TO_SOT_SMD:SOT-23, F.Cu at (85.0, -84.3)
- added Q2202: MMBT3906, Package_TO_SOT_SMD:SOT-23, F.Cu at (80.1, -84.3)
- added Q2301: MMBT3904, Package_TO_SOT_SMD:SOT-23, F.Cu at (102.5, -62.0)
- added Q2302: MMBT3906, Package_TO_SOT_SMD:SOT-23, F.Cu at (97.6, -62.0)
- added Q2401: MMBT3904, Package_TO_SOT_SMD:SOT-23, F.Cu at (120.1, -73.2)
- added Q2402: MMBT3906, Package_TO_SOT_SMD:SOT-23, F.Cu at (115.2, -73.2)
- added Q2501: MMBT3904, Package_TO_SOT_SMD:SOT-23, F.Cu at (67.5, -39.7)
- added Q2502: MMBT3906, Package_TO_SOT_SMD:SOT-23, F.Cu at (62.6, -39.7)
- added Q2601: MMBT3904, Package_TO_SOT_SMD:SOT-23, F.Cu at (102.5, -39.7)
- added Q2602: MMBT3906, Package_TO_SOT_SMD:SOT-23, F.Cu at (97.6, -39.7)
- added Q2701: MMBT3904, Package_TO_SOT_SMD:SOT-23, F.Cu at (120.1, -50.8)
- added Q2702: MMBT3906, Package_TO_SOT_SMD:SOT-23, F.Cu at (115.2, -50.8)
- added Q2801: MMBT3904, Package_TO_SOT_SMD:SOT-23, F.Cu at (102.5, -50.8)
- added Q2802: MMBT3906, Package_TO_SOT_SMD:SOT-23, F.Cu at (97.6, -50.8)
- added Q801: MMBT3904, Package_TO_SOT_SMD:SOT-23, F.Cu at (85.0, -62.0)
- added Q802: MMBT3906, Package_TO_SOT_SMD:SOT-23, F.Cu at (80.1, -62.0)
- added Q901: MMBT3904, Package_TO_SOT_SMD:SOT-23, F.Cu at (85.0, -39.7)
- added Q902: MMBT3906, Package_TO_SOT_SMD:SOT-23, F.Cu at (80.1, -39.7)
- added R1001: 10K, Resistor_SMD:R_0805_2012Metric, F.Cu at (79.9, -47.1)
- added R1002: 2K2, Resistor_SMD:R_0805_2012Metric, F.Cu at (89.7, -51.6)
- added R1003: 250R, Resistor_SMD:R_0805_2012Metric, F.Cu at (84.3, -47.1)
- added R1101: 10K, Resistor_SMD:R_0805_2012Metric, F.Cu at (79.9, -69.5)
- added R1102: 2K2, Resistor_SMD:R_0805_2012Metric, F.Cu at (89.7, -73.9)
- added R1103: 250R, Resistor_SMD:R_0805_2012Metric, F.Cu at (84.3, -69.5)
- added R1201: 10K, Resistor_SMD:R_0805_2012Metric, F.Cu at (62.3, -80.6)
- added R1202: 2K2, Resistor_SMD:R_0805_2012Metric, F.Cu at (72.1, -85.1)
- added R1203: 250R, Resistor_SMD:R_0805_2012Metric, F.Cu at (66.8, -80.6)
- added R1301: 10K, Resistor_SMD:R_0805_2012Metric, F.Cu at (132.5, -69.5)
- added R1302: 2K2, Resistor_SMD:R_0805_2012Metric, F.Cu at (142.2, -73.9)
- added R1303: 250R, Resistor_SMD:R_0805_2012Metric, F.Cu at (136.9, -69.5)
- added R1401: 10K, Resistor_SMD:R_0805_2012Metric, F.Cu at (62.3, -69.5)
- added R1402: 2K2, Resistor_SMD:R_0805_2012Metric, F.Cu at (72.1, -73.9)
- added R1403: 250R, Resistor_SMD:R_0805_2012Metric, F.Cu at (66.8, -69.5)
- added R1501: 10K, Resistor_SMD:R_0805_2012Metric, F.Cu at (62.3, -58.3)
- added R1502: 2K2, Resistor_SMD:R_0805_2012Metric, F.Cu at (72.1, -62.8)
- added R1503: 250R, Resistor_SMD:R_0805_2012Metric, F.Cu at (66.8, -58.3)
- added R1601: 10K, Resistor_SMD:R_0805_2012Metric, F.Cu at (97.4, -69.5)
- added R1602: 2K2, Resistor_SMD:R_0805_2012Metric, F.Cu at (107.2, -73.9)
- added R1603: 250R, Resistor_SMD:R_0805_2012Metric, F.Cu at (101.8, -69.5)
- added R1701: 10K, Resistor_SMD:R_0805_2012Metric, F.Cu at (114.9, -80.6)
- added R1702: 2K2, Resistor_SMD:R_0805_2012Metric, F.Cu at (124.7, -85.1)
- added R1703: 250R, Resistor_SMD:R_0805_2012Metric, F.Cu at (119.3, -80.6)
- added R1801: 10K, Resistor_SMD:R_0805_2012Metric, F.Cu at (132.5, -80.6)
- added R1802: 2K2, Resistor_SMD:R_0805_2012Metric, F.Cu at (142.2, -85.1)
- added R1803: 250R, Resistor_SMD:R_0805_2012Metric, F.Cu at (136.9, -80.6)
- added R1901: 10K, Resistor_SMD:R_0805_2012Metric, F.Cu at (114.9, -58.3)
- added R1902: 2K2, Resistor_SMD:R_0805_2012Metric, F.Cu at (124.7, -62.8)
- added R1903: 250R, Resistor_SMD:R_0805_2012Metric, F.Cu at (119.3, -58.3)
- added R2001: 10K, Resistor_SMD:R_0805_2012Metric, F.Cu at (97.4, -80.6)
- added R2002: 2K2, Resistor_SMD:R_0805_2012Metric, F.Cu at (107.2, -85.1)
- added R2003: 250R, Resistor_SMD:R_0805_2012Metric, F.Cu at (101.8, -80.6)
- added R2101: 10K, Resistor_SMD:R_0805_2012Metric, F.Cu at (62.3, -47.1)
- added R2102: 2K2, Resistor_SMD:R_0805_2012Metric, F.Cu at (72.1, -51.6)
- added R2103: 250R, Resistor_SMD:R_0805_2012Metric, F.Cu at (66.8, -47.1)
- added R2201: 10K, Resistor_SMD:R_0805_2012Metric, F.Cu at (79.9, -80.6)
- added R2202: 2K2, Resistor_SMD:R_0805_2012Metric, F.Cu at (89.7, -85.1)
- added R2203: 250R, Resistor_SMD:R_0805_2012Metric, F.Cu at (84.3, -80.6)
- added R2301: 10K, Resistor_SMD:R_0805_2012Metric, F.Cu at (97.4, -58.3)
- added R2302: 2K2, Resistor_SMD:R_0805_2012Metric, F.Cu at (107.2, -62.8)
- added R2303: 250R, Resistor_SMD:R_0805_2012Metric, F.Cu at (101.8, -58.3)
- added R2401: 10K, Resistor_SMD:R_0805_2012Metric, F.Cu at (114.9, -69.5)
- added R2402: 2K2, Resistor_SMD:R_0805_2012Metric, F.Cu at (124.7, -73.9)
- added R2403: 250R, Resistor_SMD:R_0805_2012Metric, F.Cu at (119.3, -69.5)
- added R2501: 10K, Resistor_SMD:R_0805_2012Metric, F.Cu at (62.3, -36.0)
- added R2502: 2K2, Resistor_SMD:R_0805_2012Metric, F.Cu at (72.1, -40.4)
- added R2503: 250R, Resistor_SMD:R_0805_2012Metric, F.Cu at (66.8, -36.0)
- added R2601: 10K, Resistor_SMD:R_0805_2012Metric, F.Cu at (97.4, -36.0)
- added R2602: 2K2, Resistor_SMD:R_0805_2012Metric, F.Cu at (107.2, -40.4)
- added R2603: 250R, Resistor_SMD:R_0805_2012Metric, F.Cu at (101.8, -36.0)
- added R2701: 10K, Resistor_SMD:R_0805_2012Metric, F.Cu at (114.9, -47.1)
- added R2702: 2K2, Resistor_SMD:R_0805_2012Metric, F.Cu at (124.7, -51.6)
- added R2703: 250R, Resistor_SMD:R_0805_2012Metric, F.Cu at (119.3, -47.1)
- added R2801: 10K, Resistor_SMD:R_0805_2012Metric, F.Cu at (97.4, -47.1)
- added R2802: 2K2, Resistor_SMD:R_0805_2012Metric, F.Cu at (107.2, -51.6)
- added R2803: 250R, Resistor_SMD:R_0805_2012Metric, F.Cu at (101.8, -47.1)
- added R801: 10K, Resistor_SMD:R_0805_2012Metric, F.Cu at (79.9, -58.3)
- added R802: 2K2, Resistor_SMD:R_0805_2012Metric, F.Cu at (89.7, -62.8)
- added R803: 250R, Resistor_SMD:R_0805_2012Metric, F.Cu at (84.3, -58.3)
- added R901: 10K, Resistor_SMD:R_0805_2012Metric, F.Cu at (79.9, -36.0)
- added R902: 2K2, Resistor_SMD:R_0805_2012Metric, F.Cu at (89.7, -40.4)
- added R903: 250R, Resistor_SMD:R_0805_2012Metric, F.Cu at (84.3, -36.0)
- moved U701 46.8 mm to (139.5, 133.2)
- moved U501 45.7 mm to (71.8, 133.2)
- moved U601 0.79 mm to (104.8, 133.2)

Commit message: With thanks to @ka2qfx
Parts:
- removed C601, C701: 10uF, Capacitor_SMD:C_0805_2012Metric
- removed the J102 at (91.5, 127.2)
- removed J103, J105: OUT, Connector_PinSocket_2.54mm:PinSocket_1x06_P2.54mm_Vertical
- removed J104: IN, Connector_PinSocket_2.54mm:PinSocket_1x06_P2.54mm_Vertical
- removed J601, J701: Top Conn, Connector_PinSocket_2.54mm:PinSocket_1x09_P2.54mm_Vertical
- removed J602, J702: Bottom Conn, Connector_PinSocket_2.54mm:PinSocket_1x09_P2.54mm_Vertical
- removed Q1301, Q1401, Q1501, Q1601, Q1701, Q1801, Q1901, Q2001, Q2101, Q2201, Q2301, Q2401, Q2501, Q2601, Q2701, Q2801, Q501: MMBT3904, Package_TO_SOT_SMD:SOT-23
- removed Q1302, Q1402, Q1502, Q1602, Q1702, Q1802, Q1902, Q2002, Q2102, Q2202, Q2302, Q2402, Q2502, Q2602, Q2702, Q2802: MMBT3906, Package_TO_SOT_SMD:SOT-23
- removed R1301, R1401, R1501, R1601, R1701, R1801, R1901, R2001, R2101, R2201, R2301, R2401, R2501, R2601, R2701, R2801, R501: 10K, Resistor_SMD:R_0805_2012Metric
- removed R1302, R1402, R1502, R1602, R1702, R1802, R1902, R2002, R2102, R2202, R2302, R2402, R2502, R2602, R2702, R2802: 2K2, Resistor_SMD:R_0805_2012Metric
- removed R1303, R1403, R1503, R1603, R1703, R1803, R1903, R2003, R2103, R2203, R2303, R2403, R2503, R2603, R2703, R2803: 250R, Resistor_SMD:R_0805_2012Metric
- removed U601, U701: SN74HC595, KenwoodFox:SN74HC595
- removed mouse-bite-3mm-slot (x4): VAL**, Panelization:mouse-bite-3mm-slot
- added J101: IN, Connector_PinSocket_2.54mm:PinSocket_1x06_P2.54mm_Vertical, F.Cu at (110.5, 128.2)
- added Q602: MMBT3906, Package_TO_SOT_SMD:SOT-23, F.Cu at (157.5, 123.0)
- added Q702: MMBT3906, Package_TO_SOT_SMD:SOT-23, F.Cu at (157.4, 114.5)
- added R602: 2K2, Resistor_SMD:R_0805_2012Metric, F.Cu at (159.5, 120.0)
- added R603: 250R, Resistor_SMD:R_0805_2012Metric, F.Cu at (156.0, 120.0)
- added R702: 2K2, Resistor_SMD:R_0805_2012Metric, F.Cu at (159.4, 111.5)
- added R703: 250R, Resistor_SMD:R_0805_2012Metric, F.Cu at (155.9, 111.5)
- J501: value Top Conn -> Bottom Conn
- J502: value Bottom Conn -> Top Conn
- moved U202 353.5 mm to (113.0, 54.0), turned to -90 degrees
- moved R205 347.5 mm to (117.0, 58.0), turned to -90 degrees
- moved BT201 324.9 mm to (119.5, 38.0), turned to -90 degrees
- moved R204 317.4 mm to (119.0, 58.0), turned to -90 degrees
- moved D201 307.2 mm to (149.5, 105.1), turned to -90 degrees
- moved Q601 305.5 mm to (161.1, 123.0), turned to -90 degrees
- moved Q701 305.3 mm to (161.0, 114.5), turned to -90 degrees
- moved R601 305.0 mm to (163.0, 120.0), turned to 180 degrees
- moved R701 304.9 mm to (162.9, 111.5), turned to 180 degrees
- moved R203 302.0 mm to (149.5, 101.6), turned to -90 degrees
- moved G*** 282.7 mm to (118.5, 156.5)
- moved J301 281.0 mm to (115.1, 114.0), turned to -90 degrees
- moved J302 274.6 mm to (124.5, 114.0), turned to 180 degrees
- moved C301 274.2 mm to (123.0, 128.0)
- moved C302 272.4 mm to (115.0, 105.5), turned to 90 degrees
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- renumbered J101 to J102, R202 to R201, R203 to R202, R204 to R203, R205 to R204, R206 to R205, R201 to R206
Connections:
- net /Display Card 0/CLOCK_IN renamed /C_OUT
- net /Display Card 0/DATA_IN renamed /D_OUT
- net /Display Card 0/DATA_OUT renamed /Display Card/DATA_OUT
- net /Display Card 0/LATCH_IN renamed /L_OUT
- net Net-(J301-Pad2) renamed /USB/USB-
- net Net-(J301-Pad3) renamed /USB/USB+
- J501 pad 1: /Display Card 0/SEG_B_LAMP -> unconnected-(J501-Pad1)
- J501 pad 3: /Display Card 0/SEG_A_LAMP -> /Display Card/SEG_C_LAMP
- J501 pad 5: GND -> /Display Card/SEG_D_LAMP
- J501 pad 7: /Display Card 0/SEG_F_LAMP -> /Display Card/SEG_E_LAMP
- J501 pad 9: /Display Card 0/SEG_G_LAMP -> GND
- J502 pad 1: unconnected-(J502-Pad1) -> /Display Card/SEG_B_LAMP
- J502 pad 3: /Display Card 0/SEG_C_LAMP -> /Display Card/SEG_A_LAMP
- J502 pad 5: /Display Card 0/SEG_D_LAMP -> GND
- J502 pad 7: /Display Card 0/SEG_E_LAMP -> /Display Card/SEG_F_LAMP
- J502 pad 9: GND -> /Display Card/SEG_G_LAMP
- Q601 pad 1: /Display Card 1/SEG_B -> Net-(Q601-Pad1)
- Q701 pad 1: /Display Card 2/SEG_B -> Net-(Q701-Pad1)
- R1001 pad 1: /Display Card 2/SEG_A -> /Display Card/SEG_G
- R1003 pad 2: /Display Card 2/SEG_A_LAMP -> /Display Card/SEG_G_LAMP
- R1101 pad 1: /Display Card 0/SEG_B -> /Display Card/SEG_F
- R1103 pad 2: /Display Card 0/SEG_B_LAMP -> /Display Card/SEG_F_LAMP
- R1201 pad 1: /Display Card 1/SEG_B -> /Display Card/SEG_E
- R1203 pad 2: /Display Card 1/SEG_B_LAMP -> /Display Card/SEG_E_LAMP
- R601 pad 1: /Display Card 1/SEG_B -> /Display Card/SEG_A
- R601 pad 2: GND -> Net-(Q601-Pad1)
- R701 pad 1: /Display Card 2/SEG_B -> /Display Card/SEG_B
- R701 pad 2: GND -> Net-(Q701-Pad1)
- R801 pad 1: /Display Card 0/SEG_A -> /Display Card/SEG_D
- R803 pad 2: /Display Card 0/SEG_A_LAMP -> /Display Card/SEG_D_LAMP
- R901 pad 1: /Display Card 1/SEG_A -> /Display Card/SEG_C
- R903 pad 2: /Display Card 1/SEG_A_LAMP -> /Display Card/SEG_C_LAMP
- U501 pad 1: /Display Card 0/SEG_B -> /Display Card/SEG_B
- U501 pad 15: /Display Card 0/SEG_A -> /Display Card/SEG_A
- U501 pad 2: /Display Card 0/SEG_C -> /Display Card/SEG_C
- U501 pad 3: /Display Card 0/SEG_D -> /Display Card/SEG_D
- U501 pad 4: /Display Card 0/SEG_E -> /Display Card/SEG_E
- U501 pad 5: /Display Card 0/SEG_F -> /Display Card/SEG_F
- U501 pad 6: /Display Card 0/SEG_G -> /Display Card/SEG_G
Routing:
- net +5V: track 0.00 -> 303.3 mm, vias 0 -> 14
- net +19V: track 0.00 -> 215.8 mm, vias 0 -> 8
- net /L_OUT: track 0.00 -> 99.1 mm, vias 0 -> 2
- net /C_OUT: track 0.00 -> 92.7 mm, vias 0 -> 2
- net /Display Card/SEG_A_LAMP: track 0.00 -> 90.3 mm, vias 0 -> 1
- net /Display Card/SEG_B_LAMP: track 0.00 -> 86.9 mm, vias 0 -> 2
- net /MCU/SCL: track 0.00 -> 84.2 mm
- net /D_OUT: track 0.00 -> 82.8 mm, vias 0 -> 3
- net /Display Card/SEG_E_LAMP: track 0.00 -> 82.2 mm, vias 0 -> 1
- net /Display Card/SEG_G: track 0.00 -> 74.3 mm
- net /MCU/SDA: track 0.00 -> 72.7 mm
- net /Display Card/SEG_D_LAMP: track 0.00 -> 69.8 mm, vias 0 -> 1
- net /Display Card/SEG_F: track 0.00 -> 65.3 mm
- net /MCU/DAY_RESET: track 0.00 -> 64.6 mm, vias 0 -> 1
- net /Display Card/SEG_C_LAMP: track 0.00 -> 59.3 mm
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Other:
- board size 114.5 x 141 mm -> 64.4 x 141 mm
- board text added: "LCD Display Card ${FULL_VERSION}"
