File: Hardware/days_worked_counter/mcu.kicad_sch (KiCad schematic)
At the start: 9 parts, among them SW201 RESET, U201 ATmega328P-A, Y201 16mhz

Commit message: Cleanup more stuff
Parts:
- added D201: STAT, symbol Device:LED
- added R204: 1K, Resistor_SMD:R_0805_2012Metric, symbol Device:R_Small
Connections:
- net GND: now also R204.1
- net DATA_OUT: now reaches U201.12 (PB0)
- net CLOCK_OUT: now reaches U201.13 (PB1)
- net LATCH_OUT: now reaches U201.14 (PB2)
- net at U201.17 (PB5): now also D201.2 (A)
- net DAY_RESET: now reaches U201.23 (PC0)
- net DAY_ADVANCE: now reaches U201.24 (PC1)
- net DAY_SUBTRACT: now reaches U201.25 (PC2)
- new net: D201.1 (K), R204.2
- no-connect marks 2 -> 13
Other:
- moved on the sheet: Y201
Changed lines of the file:
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@@
   (junction (at 85.09 54.61) (diameter 0) (color 0 0 0 0)
   )
+  (no_connect (at 118.11 116.84))
+  (no_connect (at 118.11 91.44))
+  (no_connect (at 118.11 93.98))
   (no_connect (at 87.63 68.58))
+  (no_connect (at 118.11 114.3))
+  (no_connect (at 118.11 96.52))
+  (no_connect (at 118.11 109.22))
+  (no_connect (at 118.11 111.76))
+  (no_connect (at 118.11 71.12))
+  (no_connect (at 118.11 119.38))
+  (no_connect (at 118.11 121.92))
   (no_connect (at 87.63 66.04))
-  (wire (pts (xy 146.05 77.47) (xy 147.32 77.47))
-    (stroke (width 0) (type default) (color 0 0 0 0))
-  )
-  (wire (pts (xy 147.32 77.47) (xy 147.32 78.74))
+  (no_connect (at 118.11 68.58))
+  (wire (pts (xy 146.05 78.74) (xy 147.32 78.74))
+    (stroke (width 0) (type default) (color 0 0 0 0))
+  )
+  (wire (pts (xy 158.75 73.66) (xy 160.02 73.66))
     (stroke (width 0) (type default) (color 0 0 0 0))
   )
@@
     (stroke (width 0) (type default) (color 0 0 0 0))
   )
-  (wire (pts (xy 137.16 74.93) (xy 138.43 74.93))
-    (stroke (width 0) (type default) (color 0 0 0 0))
-  )
   (wire (pts (xy 83.82 60.96) (xy 83.82 63.5))
     (stroke (width 0) (type default) (color 0 0 0 0))
@@
     (stroke (width 0) (type default) (color 0 0 0 0))
   )
+  (wire (pts (xy 124.46 60.96) (xy 118.11 60.96))
+    (stroke (width 0) (type default) (color 0 0 0 0))
+  )
   (wire (pts (xy 71.12 119.38) (xy 68.58 119.38))
     (stroke (width 0) (type default) (color 0 0 0 0))
   )
-  (wire (pts (xy 118.11 76.2) (xy 137.16 76.2))
+  (wire (pts (xy 118.11 76.2) (xy 138.43 76.2))
     (stroke (width 0) (type default) (color 0 0 0 0))
   )
@@
     (stroke (width 0) (type default) (color 0 0 0 0))
   )
+  (wire (pts (xy 134.62 83.82) (xy 118.11 83.82))
+    (stroke (width 0) (type default) (color 0 0 0 0))
+  )
+  (wire (pts (xy 166.37 74.93) (xy 166.37 73.66))
+    (stroke (width 0) (type default) (color 0 0 0 0))
+  )
+  (wire (pts (xy 124.46 63.5) (xy 118.11 63.5))
+    (stroke (width 0) (type default) (color 0 0 0 0))
+  )
+  (wire (pts (xy 166.37 73.66) (xy 165.1 73.66))
+    (stroke (width 0) (type default) (color 0 0 0 0))
+  )
   (wire (pts (xy 118.11 104.14) (xy 124.46 104.14))
     (stroke (width 0) (type default) (color 0 0 0 0))
@@
     (stroke (width 0) (type default) (color 0 0 0 0))
   )
+  (wire (pts (xy 118.11 73.66) (xy 151.13 73.66))
+    (stroke (width 0) (type default) (color 0 0 0 0))
+  )
+  (wire (pts (xy 134.62 88.9) (xy 118.11 88.9))
+    (stroke (width 0) (type default) (color 0 0 0 0))
+  )
   (wire (pts (xy 87.63 46.99) (xy 87.63 48.26))
     (stroke (width 0) (type default) (color 0 0 0 0))
@@
     (stroke (width 0) (type default) (color 0 0 0 0))
   )
-  (wire (pts (xy 137.16 76.2) (xy 137.16 74.93))
-    (stroke (width 0) (type default) (color 0 0 0 0))
-  )
   (wire (pts (xy 74.93 119.38) (xy 71.12 119.38))
     (stroke (width 0) (type default) (color 0 0 0 0))
   )
-  (wire (pts (xy 137.16 80.01) (xy 138.43 80.01))
+  (wire (pts (xy 137.16 81.28) (xy 138.43 81.28))
     (stroke (width 0) (type default) (color 0 0 0 0))
   )
@@
     (stroke (width 0) (type default) (color 0 0 0 0))
   )
+  (wire (pts (xy 134.62 86.36) (xy 118.11 86.36))
+    (stroke (width 0) (type default) (color 0 0 0 0))
+  )
   (wire (pts (xy 86.36 120.65) (xy 86.36 119.38))
     (stroke (width 0) (type default) (color 0 0 0 0))
@@
     (stroke (width 0) (type default) (color 0 0 0 0))
   )
+  (wire (pts (xy 124.46 66.04) (xy 118.11 66.04))
+    (stroke (width 0) (type default) (color 0 0 0 0))
+  )
   (wire (pts (xy 71.12 119.38) (xy 71.12 118.11))
     (stroke (width 0) (type default) (color 0 0 0 0))
@@
     (stroke (width 0) (type default) (color 0 0 0 0))
   )
-  (wire (pts (xy 137.16 78.74) (xy 137.16 80.01))
-    (stroke (width 0) (type default) (color 0 0 0 0))
+  (wire (pts (xy 137.16 78.74) (xy 137.16 81.28))
+    (stroke (width 0) (type default) (color 0 0 0 0))
+  )
+  (label "DAY_ADVANCE" (at 134.62 86.36 180)
+    (effects (font (size 1.27 1.27)) (justify right bottom))
+  )
+  (label "DAY_SUBTRACT" (at 134.62 88.9 180)
+    (effects (font (size 1.27 1.27)) (justify right bottom))
+  )
+  (label "DAY_RESET" (at 134.62 83.82 180)
+    (effects (font (size 1.27 1.27)) (justify right bottom))
   )
   (hierarchical_label "RST" (shape input) (at 120.65 99.06 0)
@@
   )
   (hierarchical_label "RXD" (shape input) (at 135.89 104.14 0)
+    (effects (font (size 1.27 1.27)) (justify left))
+  )
+  (hierarchical_label "CLOCK_OUT" (shape output) (at 124.46 63.5 0)
+    (effects (font (size 1.27 1.27)) (justify left))
+  )
+  (hierarchical_label "DATA_OUT" (shape output) (at 124.46 60.96 0)
+    (effects (font (size 1.27 1.27)) (justify left))
+  )
+  (hierarchical_label "LATCH_OUT" (shape output) (at 124.46 66.04 0)
     (effects (font (size 1.27 1.27)) (justify left))
   )
@@
     )
     (pin "1")
+  )
+  (symbol (lib_id "Device:LED") (at 154.94 73.66 180) (unit 1)
+    (in_bom yes) (on_board yes)
+    (property "Reference" "D201" (id 0) (at 154.94 67.31 0))
+    (property "Value" "STAT" (id 1) (at 154.94 69.85 0))
+    (property "Footprint" "" (id 2) (at 154.94 73.66 0)
+      (effects (font (size 1.27 1.27)) hide)
+    )
+    (property "Datasheet" "~" (id 3) (at 154.94 73.66 0)
+      (effects (font (size 1.27 1.27)) hide)
+    )
+    (pin "1")
+    (pin "2")
   )
   (symbol (lib_id "power:+5V") (at 85.09 46.99 0) (unit 1)
@@
     (pin "1")
   )
+  (symbol (lib_id "Device:R_Small") (at 162.56 73.66 270) (unit 1)
+    (in_bom yes) (on_board yes)
+    (property "Reference" "R204" (id 0) (at 162.56 68.58 90))
+    (property "Value" "1K" (id 1) (at 162.56 71.12 90))
+    (property "Footprint" "Resistor_SMD:R_0805_2012Metric" (id 2) (at 162.56 73.66 0)
+      (effects (font (size 1.27 1.27)) hide)
+    )
+    (property "Datasheet" "~" (id 3) (at 162.56 73.66 0)
+      (effects (font (size 1.27 1.27)) hide)
+    )
+    (pin "1")
+    (pin "2")
+  )
   (symbol (lib_id "Switch:SW_Push") (at 80.01 119.38 0) (unit 1)
     (in_bom yes) (on_board yes)
@@
     (pin "2")
   )
-  (symbol (lib_id "Device:Resonator_Small") (at 140.97 77.47 90) (unit 1)
-    (in_bom yes) (on_board yes) (fields_autoplaced)
-    (property "Reference" "Y201" (id 0) (at 141.9733 68.58 90))
-    (property "Value" "16mhz" (id 1) (at 141.9733 71.12 90))
-    (property "Footprint" "" (id 2) (at 140.97 78.105 0)
-      (effects (font (size 1.27 1.27)) hide)
-    )
-    (property "Datasheet" "~" (id 3) (at 140.97 78.105 0)
+  (symbol (lib_id "Device:Resonator_Small") (at 140.97 78.74 90) (unit 1)
+    (in_bom yes) (on_board yes)
+    (property "Reference" "Y201" (id 0) (at 139.7 83.82 90))
+    (property "Value" "16mhz" (id 1) (at 139.7 86.36 90))
+    (property "Footprint" "" (id 2) (at 140.97 79.375 0)
+      (effects (font (size 1.27 1.27)) hide)
+    )
+    (property "Datasheet" "~" (id 3) (at 140.97 79.375 0)
       (effects (font (size 1.27 1.27)) hide)
     )
@@
       (effects (font (size 1.27 1.27)) hide)
     )
+    (pin "1")
+  )
+  (symbol (lib_id "power:GND") (at 166.37 74.93 0) (unit 1)
+    (in_bom yes) (on_board yes)
+    (property "Reference" "#PWR0143" (id 0) (at 166.37 81.28 0)
+      (effects (font (size 1.27 1.27)) hide)
+    )
+    (property "Value" "GND" (id 1) (at 166.37 78.74 0))
+    (property "Footprint" "" (id 2) (at 166.37 74.93 0)
+      (effects (font (size 1.27 1.27)) hide)
+    )
+    (property "Datasheet" "" (id 3) (at 166.37 74.93 0)
+      (effects (font (size 1.27 1.27)) hide)
+    )

Commit message: Add all the cool stuff
Other:
- company: (none) -> FRC 1721
- title: (none) -> Days Without Incident Sign
Changed lines of the file:
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@@
 (kicad_sch (version 20211123) (generator eeschema)
   (paper "A4")
+  (title_block
+    (title "Days Without Incident Sign")
+    (date "2022-06-24")
+    (rev "v0.1-RC1")
+    (company "FRC 1721")
+  )
   (junction (at 71.12 119.38) (diameter 0) (color 0 0 0 0)
   )

Commit message: Even more stuff
Parts:
- added BT201: 3v, Battery:BatteryHolder_Keystone_3034_1x20mm, symbol Device:Battery_Cell
- added R205, R206: 10K, Resistor_SMD:R_0805_2012Metric, symbol Device:R_Small
- added U202: DS1307Z+, Package_SO:SOIC-8_3.9x4.9mm_P1.27mm, symbol Timer_RTC:DS1307Z+
- added Y202: 32.768kHz, symbol Device:Crystal
- D201: footprint (none) -> LED_SMD:LED_0805_2012Metric
Connections:
- net +5V: now also R205.1, R206.1, U202.8 (VCC)
- net GND: now also BT201.2 (-), U202.4 (GND)
- net SDA: now reaches U201.27 (PC4)
- net SDA: now also R206.2, U202.5 (SDA)
- net SCL: now reaches U201.28 (PC5)
- net SCL: now also R205.2, U202.6 (SCL)
- new net: BT201.1 (+), U202.3 (VBAT)
- new net: U202.1 (X1), Y202.2
- new net: U202.2 (X2), Y202.1
- no-connect marks 13 -> 12

Commit message: get input from @ka2qfx
Parts:
- removed Y201: 16mhz, symbol Device:Resonator_Small
- added C204, C205: 22pf, Capacitor_SMD:C_0805_2012Metric, symbol Device:C_Small
- added R207, R208, R209: 10K, Resistor_SMD:R_0805_2012Metric, symbol Device:R_Small
- added SW202: DAY_RESET, Button_Switch_THT:SW_PUSH_6mm_H5mm, symbol Switch:SW_Push
- added SW203: DAY_ADV, Button_Switch_THT:SW_PUSH_6mm_H5mm, symbol Switch:SW_Push
- added SW204: DAY_SUB, Button_Switch_THT:SW_PUSH_6mm_H5mm, symbol Switch:SW_Push
- added Y201: 16mHz, Crystal:Crystal_SMD_HC49-SD, symbol Device:Crystal
- SW201: footprint Button_Switch_SMD:SW_Push_SPST_NO_Alps_SKRK -> Button_Switch_THT:SW_PUSH_6mm_H5mm
- Y202: footprint (none) -> Crystal:Crystal_SMD_HC49-SD
Connections:
- net +5V: now also SW202.2, SW203.2, SW204.2
- net DAY_ADVANCE: now also U201.1 (PD3), R208.1, SW203.1; no longer U201.24 (PC1)
- net DAY_RESET: now also U201.32 (PD2), R207.1, SW202.1; no longer U201.23 (PC0)
- net DAY_SUBTRACT: now also U201.2 (PD4), R209.1, SW204.1; no longer U201.25 (PC2)
- net GND: now also C204.2, C205.2, R207.2, R208.2, R209.2
- net at U201.7 (XTAL1/PB6): now also C205.1, Y201.1
- net at U201.8 (XTAL2/PB7): now also C204.1, Y201.2
Other:
- note added: "16pf = (22pf)/2+5pf"
- moved on the sheet: BT201, C201, C202, C203, D201, R201, R202, R203, R204, R205, R206, SW201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

Commit message: With thanks to @ka2qfx
Parts:
- renumbered R202 to R201, R203 to R202, R204 to R203, R205 to R204, R206 to R205, R201 to R206
Changed lines of the file:
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@@
   (symbol (lib_id "power:+5V") (at 271.78 127.635 0) (unit 1)
     (in_bom yes) (on_board yes)
-    (property "Reference" "#PWR0204" (id 0) (at 271.78 131.445 0)
+    (property "Reference" "#PWR0218" (id 0) (at 271.78 131.445 0)
       (effects (font (size 1.27 1.27)) hide)
     )
@@
   (symbol (lib_id "Device:R_Small") (at 133.35 97.155 90) (unit 1)
     (in_bom yes) (on_board yes)
-    (property "Reference" "R203" (id 0) (at 133.35 99.695 90))
+    (property "Reference" "R202" (id 0) (at 133.35 99.695 90))
     (property "Value" "1K" (id 1) (at 133.35 97.155 90))
     (property "Footprint" "Resistor_SMD:R_0805_2012Metric" (id 2) (at 133.35 97.155 0)
@@
   (symbol (lib_id "power:GND") (at 94.615 122.555 0) (unit 1)
     (in_bom yes) (on_board yes)
-    (property "Reference" "#PWR0106" (id 0) (at 94.615 128.905 0)
+    (property "Reference" "#PWR0204" (id 0) (at 94.615 128.905 0)
       (effects (font (size 1.27 1.27)) hide)
     )
@@
   (symbol (lib_id "power:GND") (at 247.65 44.45 0) (unit 1)
     (in_bom yes) (on_board yes)
-    (property "Reference" "#PWR0184" (id 0) (at 247.65 50.8 0)
+    (property "Reference" "#PWR0211" (id 0) (at 247.65 50.8 0)
       (effects (font (size 1.27 1.27)) hide)
     )
@@
   (symbol (lib_id "power:+5V") (at 271.78 144.145 0) (unit 1)
     (in_bom yes) (on_board yes)
-    (property "Reference" "#PWR0206" (id 0) (at 271.78 147.955 0)
+    (property "Reference" "#PWR0219" (id 0) (at 271.78 147.955 0)
       (effects (font (size 1.27 1.27)) hide)
     )
@@
   (symbol (lib_id "power:GND") (at 137.16 81.915 0) (unit 1)
     (in_bom yes) (on_board yes)
-    (property "Reference" "#PWR0103" (id 0) (at 137.16 88.265 0)
+    (property "Reference" "#PWR0206" (id 0) (at 137.16 88.265 0)
       (effects (font (size 1.27 1.27)) hide)
     )
@@
   (symbol (lib_id "power:+5V") (at 227.965 33.02 0) (unit 1)
     (in_bom yes) (on_board yes)
-    (property "Reference" "#PWR0185" (id 0) (at 227.965 36.83 0)
+    (property "Reference" "#PWR0209" (id 0) (at 227.965 36.83 0)
       (effects (font (size 1.27 1.27)) hide)
     )
@@
   (symbol (lib_id "power:+5V") (at 76.835 37.465 0) (unit 1)
     (in_bom yes) (on_board yes)
-    (property "Reference" "#PWR0101" (id 0) (at 76.835 41.275 0)
+    (property "Reference" "#PWR0202" (id 0) (at 76.835 41.275 0)
       (effects (font (size 1.27 1.27)) hide)
     )
@@
   (symbol (lib_id "Device:R_Small") (at 250.19 92.71 0) (unit 1)
     (in_bom yes) (on_board yes)
-    (property "Reference" "R201" (id 0) (at 243.84 91.44 0)
+    (property "Reference" "R206" (id 0) (at 243.84 91.44 0)
       (effects (font (size 1.27 1.27)) (justify left))
     )
@@
   (symbol (lib_id "power:GND") (at 230.505 62.23 0) (unit 1)
     (in_bom yes) (on_board yes)
-    (property "Reference" "#PWR0186" (id 0) (at 230.505 68.58 0)
+    (property "Reference" "#PWR0210" (id 0) (at 230.505 68.58 0)
       (effects (font (size 1.27 1.27)) hide)
     )
@@
   (symbol (lib_id "Device:R_Small") (at 133.35 94.615 90) (unit 1)
     (in_bom yes) (on_board yes)
-    (property "Reference" "R202" (id 0) (at 133.35 92.075 90))
+    (property "Reference" "R201" (id 0) (at 133.35 92.075 90))
     (property "Value" "1K" (id 1) (at 133.35 94.615 90))
     (property "Footprint" "Resistor_SMD:R_0805_2012Metric" (id 2) (at 133.35 94.615 0)
@@
   (symbol (lib_id "power:GND") (at 265.43 99.06 0) (unit 1)
     (in_bom yes) (on_board yes)
-    (property "Reference" "#PWR0107" (id 0) (at 265.43 105.41 0)
+    (property "Reference" "#PWR0216" (id 0) (at 265.43 105.41 0)
       (effects (font (size 1.27 1.27)) hide)
     )
@@
   (symbol (lib_id "power:+5V") (at 250.19 88.9 0) (unit 1)
     (in_bom yes) (on_board yes)
-    (property "Reference" "#PWR0108" (id 0) (at 250.19 92.71 0)
+    (property "Reference" "#PWR0212" (id 0) (at 250.19 92.71 0)
       (effects (font (size 1.27 1.27)) hide)
     )
@@
   (symbol (lib_id "Device:R_Small") (at 154.305 64.135 270) (unit 1)
     (in_bom yes) (on_board yes)
-    (property "Reference" "R204" (id 0) (at 154.305 59.055 90))
+    (property "Reference" "R203" (id 0) (at 154.305 59.055 90))
     (property "Value" "1K" (id 1) (at 154.305 61.595 90))
     (property "Footprint" "Resistor_SMD:R_0805_2012Metric" (id 2) (at 154.305 64.135 0)
@@
   (symbol (lib_id "power:+5V") (at 271.78 110.49 0) (unit 1)
     (in_bom yes) (on_board yes)
-    (property "Reference" "#PWR0202" (id 0) (at 271.78 114.3 0)
+    (property "Reference" "#PWR0217" (id 0) (at 271.78 114.3 0)
       (effects (font (size 1.27 1.27)) hide)
     )
@@
   (symbol (lib_id "power:GND") (at 75.565 61.595 0) (unit 1)
     (in_bom yes) (on_board yes) (fields_autoplaced)
-    (property "Reference" "#PWR0104" (id 0) (at 75.565 67.945 0)
+    (property "Reference" "#PWR0201" (id 0) (at 75.565 67.945 0)
       (effects (font (size 1.27 1.27)) hide)
     )
@@
   (symbol (lib_id "power:GND") (at 257.175 139.065 0) (unit 1)
     (in_bom yes) (on_board yes)
-    (property "Reference" "#PWR0207" (id 0) (at 257.175 145.415 0)
+    (property "Reference" "#PWR0214" (id 0) (at 257.175 145.415 0)
       (effects (font (size 1.27 1.27)) hide)
     )
@@
   (symbol (lib_id "power:GND") (at 257.175 121.92 0) (unit 1)
     (in_bom yes) (on_board yes)
-    (property "Reference" "#PWR0203" (id 0) (at 257.175 128.27 0)
+    (property "Reference" "#PWR0213" (id 0) (at 257.175 128.27 0)
       (effects (font (size 1.27 1.27)) hide)
     )
@@
   (symbol (lib_id "power:GND") (at 257.175 155.575 0) (unit 1)
     (in_bom yes) (on_board yes)
-    (property "Reference" "#PWR0205" (id 0) (at 257.175 161.925 0)
+    (property "Reference" "#PWR0215" (id 0) (at 257.175 161.925 0)
       (effects (font (size 1.27 1.27)) hide)
     )
@@
   (symbol (lib_id "power:+5V") (at 95.885 40.005 0) (unit 1)
     (in_bom yes) (on_board yes)
-    (property "Reference" "#PWR0102" (id 0) (at 95.885 43.815 0)
+    (property "Reference" "#PWR0205" (id 0) (at 95.885 43.815 0)
       (effects (font (size 1.27 1.27)) hide)
     )
@@
   (symbol (lib_id "power:GND") (at 76.835 45.085 0) (unit 1)
     (in_bom yes) (on_board yes)
-    (property "Reference" "#PWR0105" (id 0) (at 76.835 51.435 0)
+    (property "Reference" "#PWR0203" (id 0) (at 76.835 51.435 0)
       (effects (font (size 1.27 1.27)) hide)
     )
@@
   (symbol (lib_id "Device:R_Small") (at 206.375 41.275 0) (unit 1)
     (in_bom yes) (on_board yes)
-    (property "Reference" "R205" (id 0) (at 202.565 40.005 0))
+    (property "Reference" "R204" (id 0) (at 202.565 40.005 0))
     (property "Value" "10K" (id 1) (at 203.2 41.91 0))
     (property "Footprint" "Resistor_SMD:R_0805_2012Metric" (id 2) (at 206.375 41.275 0)
@@
   (symbol (lib_id "power:+5V") (at 210.82 33.02 0) (unit 1)
     (in_bom yes) (on_board yes)
-    (property "Reference" "#PWR0187" (id 0) (at 210.82 36.83 0)
+    (property "Reference" "#PWR0208" (id 0) (at 210.82 36.83 0)
       (effects (font (size 1.27 1.27)) hide)
     )
@@
   (symbol (lib_id "Device:R_Small") (at 215.265 41.275 0) (unit 1)
     (in_bom yes) (on_board yes)
-    (property "Reference" "R206" (id 0) (at 211.455 40.005 0))
+    (property "Reference" "R205" (id 0) (at 211.455 40.005 0))
     (property "Value" "10K" (id 1) (at 212.09 41.91 0))
     (property "Footprint" "Resistor_SMD:R_0805_2012Metric" (id 2) (at 215.265 41.275 0)
@@
   (symbol (lib_id "power:GND") (at 158.115 65.405 0) (unit 1)
     (in_bom yes) (on_board yes)
-    (property "Reference" "#PWR0143" (id 0) (at 158.115 71.755 0)
-      (effects (font (size 1.27 1.27)) hide)
-    )
+    (property "Reference" "#PWR0207" (id 0) (at 158.115 71.755 0)
+      (effects (font (size 1.27 1.27)) hide)
+    )
