File: Hardware/days_worked_counter/usb.kicad_sch (KiCad schematic)
At the start: 10 parts, among them J301 USB_B_Micro, U301 FT232RL

Commit message: Add all the cool stuff
Other:
- company: (none) -> FRC 1721
- title: (none) -> Days Without Incident Sign
Changed lines of the file:
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@@
 (kicad_sch (version 20211123) (generator eeschema)
   (paper "A4")
+  (title_block
+    (title "Days Without Incident Sign")
+    (date "2022-06-24")
+    (rev "v0.1-RC1")
+    (company "FRC 1721")
+  )
   (junction (at 105.41 76.2) (diameter 0) (color 0 0 0 0)
   )

Commit message: Even more stuff
Parts:
- added J302: PROG, Connector_PinSocket_2.54mm:PinSocket_1x06_P2.54mm_Vertical, symbol Connector:Conn_01x06_Female
- added JP301: SolderJumper_2_Open, Jumper:SolderJumper-2_P1.3mm_Open_TrianglePad1.0x1.5mm, symbol Jumper:SolderJumper_2_Open
- J301: footprint Connector_USB:USB_Micro-AB_Molex_47590-0001 -> Connector_USB:USB_Mini-B_Lumberg_2486_01_Horizontal
Connections:
- net +5V: now also JP301.1 (A)
- net GND: now also J302.6 (Pin_6)
- net RXD: now also J302.3 (Pin_3)
- net TXD: now also J302.2 (Pin_2)
- new net: J302.4 (Pin_4), JP301.2 (B)
- no-connect marks 12 -> 14
Changed lines of the file:
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@@
   (no_connect (at 124.46 93.98))
   (no_connect (at 165.1 106.68))
+  (no_connect (at 145.415 31.115))
   (no_connect (at 165.1 83.82))
   (no_connect (at 165.1 93.98))
@@
   (no_connect (at 165.1 91.44))
   (no_connect (at 165.1 109.22))
+  (no_connect (at 145.415 41.275))
   (no_connect (at 165.1 88.9))
   (no_connect (at 165.1 111.76))
@@
     (stroke (width 0) (type default) (color 0 0 0 0))
   )
+  (wire (pts (xy 144.145 36.195) (xy 145.415 36.195))
+    (stroke (width 0) (type default) (color 0 0 0 0))
+  )
+  (wire (pts (xy 142.24 38.735) (xy 145.415 38.735))
+    (stroke (width 0) (type default) (color 0 0 0 0))
+  )
   (wire (pts (xy 120.65 59.69) (xy 123.19 59.69))
     (stroke (width 0) (type default) (color 0 0 0 0))
@@
     (stroke (width 0) (type default) (color 0 0 0 0))
   )
+  (wire (pts (xy 132.08 37.465) (xy 132.08 38.735))
+    (stroke (width 0) (type default) (color 0 0 0 0))
+  )
+  (wire (pts (xy 144.145 43.815) (xy 145.415 43.815))
+    (stroke (width 0) (type default) (color 0 0 0 0))
+  )
   (wire (pts (xy 123.19 67.31) (xy 120.65 67.31))
     (stroke (width 0) (type default) (color 0 0 0 0))
@@
     (stroke (width 0) (type default) (color 0 0 0 0))
   )
+  (wire (pts (xy 144.145 33.655) (xy 145.415 33.655))
+    (stroke (width 0) (type default) (color 0 0 0 0))
+  )
   (wire (pts (xy 180.34 78.74) (xy 165.1 78.74))
     (stroke (width 0) (type default) (color 0 0 0 0))
   )
+  (wire (pts (xy 144.145 45.085) (xy 144.145 43.815))
+    (stroke (width 0) (type default) (color 0 0 0 0))
+  )
   (wire (pts (xy 82.55 109.22) (xy 81.28 109.22))
     (stroke (width 0) (type default) (color 0 0 0 0))
@@
   )
   (wire (pts (xy 139.7 119.38) (xy 139.7 121.92))
+    (stroke (width 0) (type default) (color 0 0 0 0))
+  )
+  (wire (pts (xy 132.08 38.735) (xy 134.62 38.735))
     (stroke (width 0) (type default) (color 0 0 0 0))
   )
@@
     (effects (font (size 1.27 1.27)) (justify left))
   )
+  (hierarchical_label "RXD" (shape input) (at 144.145 36.195 180)
+    (effects (font (size 1.27 1.27)) (justify right))
+  )
   (hierarchical_label "RXD" (shape input) (at 180.34 78.74 0)
     (effects (font (size 1.27 1.27)) (justify left))
+  )
+  (hierarchical_label "TXD" (shape output) (at 144.145 33.655 180)
+    (effects (font (size 1.27 1.27)) (justify right))
   )
   (symbol (lib_id "power:GND") (at 147.32 121.92 0) (unit 1)
@@
     (pin "1")
   )
+  (symbol (lib_id "power:+5V") (at 132.08 37.465 0) (unit 1)
+    (in_bom yes) (on_board yes) (fields_autoplaced)
+    (property "Reference" "#PWR0188" (id 0) (at 132.08 41.275 0)
+      (effects (font (size 1.27 1.27)) hide)
+    )
+    (property "Value" "+5V" (id 1) (at 132.08 32.385 0))
+    (property "Footprint" "" (id 2) (at 132.08 37.465 0)
+      (effects (font (size 1.27 1.27)) hide)
+    )
+    (property "Datasheet" "" (id 3) (at 132.08 37.465 0)
+      (effects (font (size 1.27 1.27)) hide)
+    )
+    (pin "1")
+  )
   (symbol (lib_id "power:VBUS") (at 92.71 90.17 0) (unit 1)
     (in_bom yes) (on_board yes)
@@
     (property "Reference" "J301" (id 0) (at 78.74 88.9 0))
     (property "Value" "USB_B_Micro" (id 1) (at 90.17 106.68 0))
-    (property "Footprint" "Connector_USB:USB_Micro-AB_Molex_47590-0001" (id 2) (at 86.36 99.06 0)
+    (property "Footprint" "Connector_USB:USB_Mini-B_Lumberg_2486_01_Horizontal" (id 2) (at 86.36 99.06 0)
       (effects (font (size 1.27 1.27)) hide)
     )
@@
     )
     (property "Datasheet" "~" (id 3) (at 105.41 80.01 0)
+      (effects (font (size 1.27 1.27)) hide)
+    )
+    (pin "1")
+    (pin "2")
+  )
+  (symbol (lib_id "Jumper:SolderJumper_2_Open") (at 138.43 38.735 0) (unit 1)
+    (in_bom yes) (on_board yes)
+    (property "Reference" "JP301" (id 0) (at 138.43 41.275 0))
+    (property "Value" "SolderJumper_2_Open" (id 1) (at 138.43 35.56 0)
+      (effects (font (size 1.27 1.27)) hide)
+    )
+    (property "Footprint" "Jumper:SolderJumper-2_P1.3mm_Open_TrianglePad1.0x1.5mm" (id 2) (at 138.43 38.735 0)
+      (effects (font (size 1.27 1.27)) hide)
+    )
+    (property "Datasheet" "~" (id 3) (at 138.43 38.735 0)
       (effects (font (size 1.27 1.27)) hide)
     )
@@
     (pin "2")
   )
+  (symbol (lib_id "Connector:Conn_01x06_Female") (at 150.495 36.195 0) (unit 1)
+    (in_bom yes) (on_board yes)
+    (property "Reference" "J302" (id 0) (at 148.59 27.94 0)
+      (effects (font (size 1.27 1.27)) (justify left))
+    )
+    (property "Value" "PROG" (id 1) (at 146.685 46.355 0)
+      (effects (font (size 1.27 1.27)) (justify left))
+    )
+    (property "Footprint" "Connector_PinSocket_2.54mm:PinSocket_1x06_P2.54mm_Vertical" (id 2) (at 150.495 36.195 0)
+      (effects (font (size 1.27 1.27)) hide)
+    )
+    (property "Datasheet" "~" (id 3) (at 150.495 36.195 0)
+      (effects (font (size 1.27 1.27)) hide)
+    )
+    (pin "1")
+    (pin "2")
+    (pin "3")
+    (pin "4")
+    (pin "5")
+    (pin "6")
+  )
   (symbol (lib_id "Device:C_Polarized_Small") (at 118.11 63.5 0) (unit 1)
     (in_bom yes) (on_board yes)
@@
       (effects (font (size 1.27 1.27)) hide)
     )
+    (pin "1")
+  )
+  (symbol (lib_id "power:GND") (at 144.145 45.085 0) (unit 1)
+    (in_bom yes) (on_board yes)
+    (property "Reference" "#PWR0189" (id 0) (at 144.145 51.435 0)
+      (effects (font (size 1.27 1.27)) hide)
+    )
+    (property "Value" "GND" (id 1) (at 144.145 48.895 0))
+    (property "Footprint" "" (id 2) (at 144.145 45.085 0)
+      (effects (font (size 1.27 1.27)) hide)
+    )
+    (property "Datasheet" "" (id 3) (at 144.145 45.085 0)
+      (effects (font (size 1.27 1.27)) hide)
+    )

Commit message: With thanks to @ka2qfx
Connections:
- net USB-: now reaches J301.2 (D-), U301.16 (USBD-)
- net USB+: now reaches J301.3 (D+), U301.15 (USBD+)
Changed lines of the file:
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@@
     (stroke (width 0) (type default) (color 0 0 0 0))
+  )
+  (label "USB+" (at 98.425 97.79 0)
+    (effects (font (size 1.27 1.27)) (justify left bottom))
+  )
+  (label "USB-" (at 98.425 100.33 0)
+    (effects (font (size 1.27 1.27)) (justify left bottom))
   )
   (hierarchical_label "RST" (shape output) (at 180.34 86.36 0)
@@
   (symbol (lib_id "power:GND") (at 147.32 121.92 0) (unit 1)
     (in_bom yes) (on_board yes)
-    (property "Reference" "#PWR0110" (id 0) (at 147.32 128.27 0)
+    (property "Reference" "#PWR0312" (id 0) (at 147.32 128.27 0)
       (effects (font (size 1.27 1.27)) hide)
     )
@@
   (symbol (lib_id "power:+5V") (at 144.78 64.77 0) (unit 1)
     (in_bom yes) (on_board yes) (fields_autoplaced)
-    (property "Reference" "#PWR0109" (id 0) (at 144.78 68.58 0)
+    (property "Reference" "#PWR0311" (id 0) (at 144.78 68.58 0)
       (effects (font (size 1.27 1.27)) hide)
     )
@@
   (symbol (lib_id "power:GND") (at 120.65 67.31 0) (unit 1)
     (in_bom yes) (on_board yes)
-    (property "Reference" "#PWR0119" (id 0) (at 120.65 73.66 0)
+    (property "Reference" "#PWR0307" (id 0) (at 120.65 73.66 0)
       (effects (font (size 1.27 1.27)) hide)
     )
@@
   (symbol (lib_id "power:+5V") (at 132.08 37.465 0) (unit 1)
     (in_bom yes) (on_board yes) (fields_autoplaced)
-    (property "Reference" "#PWR0188" (id 0) (at 132.08 41.275 0)
+    (property "Reference" "#PWR0308" (id 0) (at 132.08 41.275 0)
       (effects (font (size 1.27 1.27)) hide)
     )
@@
   (symbol (lib_id "power:VBUS") (at 92.71 90.17 0) (unit 1)
     (in_bom yes) (on_board yes)
-    (property "Reference" "#PWR0115" (id 0) (at 92.71 93.98 0)
+    (property "Reference" "#PWR0302" (id 0) (at 92.71 93.98 0)
       (effects (font (size 1.27 1.27)) hide)
     )
@@
   (symbol (lib_id "power:+5V") (at 201.93 100.33 0) (unit 1)
     (in_bom yes) (on_board yes) (fields_autoplaced)
-    (property "Reference" "#PWR0114" (id 0) (at 201.93 104.14 0)
+    (property "Reference" "#PWR0313" (id 0) (at 201.93 104.14 0)
       (effects (font (size 1.27 1.27)) hide)
     )
@@
   (symbol (lib_id "power:VBUS") (at 120.65 59.69 0) (unit 1)
     (in_bom yes) (on_board yes)
-    (property "Reference" "#PWR0113" (id 0) (at 120.65 63.5 0)
+    (property "Reference" "#PWR0306" (id 0) (at 120.65 63.5 0)
       (effects (font (size 1.27 1.27)) hide)
     )
@@
   (symbol (lib_id "power:GND") (at 105.41 83.82 0) (unit 1)
     (in_bom yes) (on_board yes)
-    (property "Reference" "#PWR0116" (id 0) (at 105.41 90.17 0)
+    (property "Reference" "#PWR0304" (id 0) (at 105.41 90.17 0)
       (effects (font (size 1.27 1.27)) hide)
     )
@@
   (symbol (lib_id "power:GND") (at 139.7 121.92 0) (unit 1)
     (in_bom yes) (on_board yes)
-    (property "Reference" "#PWR0111" (id 0) (at 139.7 128.27 0)
+    (property "Reference" "#PWR0309" (id 0) (at 139.7 128.27 0)
       (effects (font (size 1.27 1.27)) hide)
     )
@@
   (symbol (lib_id "power:+3.3V") (at 105.41 74.93 0) (unit 1)
     (in_bom yes) (on_board yes)
-    (property "Reference" "#PWR0118" (id 0) (at 105.41 78.74 0)
+    (property "Reference" "#PWR0303" (id 0) (at 105.41 78.74 0)
       (effects (font (size 1.27 1.27)) hide)
     )
@@
   (symbol (lib_id "power:GND") (at 81.28 110.49 0) (unit 1)
     (in_bom yes) (on_board yes)
-    (property "Reference" "#PWR0117" (id 0) (at 81.28 116.84 0)
+    (property "Reference" "#PWR0301" (id 0) (at 81.28 116.84 0)
       (effects (font (size 1.27 1.27)) hide)
     )
@@
   (symbol (lib_id "power:GND") (at 119.38 121.92 0) (unit 1)
     (in_bom yes) (on_board yes)
-    (property "Reference" "#PWR0112" (id 0) (at 119.38 128.27 0)
+    (property "Reference" "#PWR0305" (id 0) (at 119.38 128.27 0)
       (effects (font (size 1.27 1.27)) hide)
     )
@@
   (symbol (lib_id "power:GND") (at 144.145 45.085 0) (unit 1)
     (in_bom yes) (on_board yes)
-    (property "Reference" "#PWR0189" (id 0) (at 144.145 51.435 0)
-      (effects (font (size 1.27 1.27)) hide)
-    )
+    (property "Reference" "#PWR0310" (id 0) (at 144.145 51.435 0)
+      (effects (font (size 1.27 1.27)) hide)
+    )
