File: Hardware/Segment_Display_Board/mcu.kicad_sch (KiCad schematic)
At the start: 24 parts, among them SW201 RESET, SW202 DAY_RESET, SW203 DAY_ADV, SW204 DAY_SUB, U201 ATmega328P-A, U202 DS1307Z+, Y201 16mHz, Y202 32.768kHz

Commit message: Fix stuff i guess goodnight"
Changed lines of the file:
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@@
     (title "Days Without Incident Sign")
     (date "2022-06-24")
-    (rev "v0.1-RC1")
+    (rev "${REVISION}")
     (company "FRC 1721")
+    (comment 4 "Release: ${FULL_REVISION}")
   )
   (junction (at 250.19 97.79) (diameter 0) (color 0 0 0 0)
@@
   )
   (junction (at 76.835 37.465) (diameter 0) (color 0 0 0 0)
+  )
+  (junction (at 247.65 33.655) (diameter 0) (color 0 0 0 0)
   )
   (junction (at 257.175 130.175) (diameter 0) (color 0 0 0 0)
@@
     (pin "2")
   )
+  (symbol (lib_id "power:PWR_FLAG") (at 247.65 33.655 0) (unit 1)
+    (in_bom yes) (on_board yes) (fields_autoplaced)
+    (property "Reference" "#FLG0201" (id 0) (at 247.65 31.75 0)
+      (effects (font (size 1.27 1.27)) hide)
+    )
+    (property "Value" "PWR_FLAG" (id 1) (at 247.65 27.94 0)
+      (effects (font (size 1.27 1.27)) hide)
+    )
+    (property "Footprint" "" (id 2) (at 247.65 33.655 0)
+      (effects (font (size 1.27 1.27)) hide)
+    )
+    (property "Datasheet" "~" (id 3) (at 247.65 33.655 0)
+      (effects (font (size 1.27 1.27)) hide)
+    )
+    (pin "1")
+  )
   (symbol (lib_id "Device:C_Polarized_Small") (at 74.295 41.275 0) (unit 1)

Commit message: Place hardware orders
Parts:
- Y202: footprint Crystal:Crystal_SMD_HC49-SD -> Crystal:Crystal_C38-LF_D3.0mm_L8.0mm_Horizontal
Changed lines of the file:
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@@
       (effects (font (size 1.27 1.27)) (justify right))
     )
-    (property "Footprint" "Crystal:Crystal_SMD_HC49-SD" (id 2) (at 205.74 54.61 0)
+    (property "Footprint" "Crystal:Crystal_C38-LF_D3.0mm_L8.0mm_Horizontal" (id 2) (at 205.74 54.61 0)
       (effects (font (size 1.27 1.27)) hide)
     )

Commit message: include fixups fro EE
Parts:
- removed C201: 4.7uf, Capacitor_SMD:CP_Elec_4x3, symbol Device:C_Polarized_Small
- renumbered C202 to C201, C203 to C202, C204 to C203, C205 to C204
Other:
- moved on the sheet: C202
Changed lines of the file:
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@@
   (junction (at 95.885 42.545) (diameter 0) (color 0 0 0 0)
   )
-  (junction (at 76.835 37.465) (diameter 0) (color 0 0 0 0)
-  )
   (junction (at 247.65 33.655) (diameter 0) (color 0 0 0 0)
   )
@@
   )
   (junction (at 132.715 72.39) (diameter 0) (color 0 0 0 0)
-  )
-  (junction (at 76.835 45.085) (diameter 0) (color 0 0 0 0)
   )
   (junction (at 137.16 81.28) (diameter 0) (color 0 0 0 0)
@@
     (stroke (width 0) (type default) (color 0 0 0 0))
   )
-  (wire (pts (xy 74.295 37.465) (xy 74.295 38.735))
-    (stroke (width 0) (type default) (color 0 0 0 0))
-  )
   (wire (pts (xy 109.855 97.155) (xy 130.81 97.155))
     (stroke (width 0) (type default) (color 0 0 0 0))
@@
     (stroke (width 0) (type default) (color 0 0 0 0))
   )
-  (wire (pts (xy 79.375 45.085) (xy 76.835 45.085))
-    (stroke (width 0) (type default) (color 0 0 0 0))
-  )
   (wire (pts (xy 257.175 153.67) (xy 257.175 155.575))
     (stroke (width 0) (type default) (color 0 0 0 0))
   )
-  (wire (pts (xy 79.375 43.815) (xy 79.375 45.085))
+  (wire (pts (xy 90.17 38.1) (xy 90.17 39.37))
     (stroke (width 0) (type default) (color 0 0 0 0))
   )
@@
     (stroke (width 0) (type default) (color 0 0 0 0))
   )
-  (wire (pts (xy 79.375 37.465) (xy 79.375 38.735))
+  (wire (pts (xy 90.17 31.75) (xy 90.17 33.02))
     (stroke (width 0) (type default) (color 0 0 0 0))
   )
@@
     (stroke (width 0) (type default) (color 0 0 0 0))
   )
-  (wire (pts (xy 76.835 37.465) (xy 79.375 37.465))
-    (stroke (width 0) (type default) (color 0 0 0 0))
-  )
   (wire (pts (xy 230.505 60.96) (xy 230.505 62.23))
     (stroke (width 0) (type default) (color 0 0 0 0))
@@
     (stroke (width 0) (type default) (color 0 0 0 0))
   )
-  (wire (pts (xy 76.835 45.085) (xy 74.295 45.085))
-    (stroke (width 0) (type default) (color 0 0 0 0))
-  )
   (polyline (pts (xy 177.165 75.565) (xy 285.115 75.565))
     (stroke (width 0) (type default) (color 0 0 0 0))
@@
     (stroke (width 0) (type default) (color 0 0 0 0))
   )
-  (wire (pts (xy 74.295 45.085) (xy 74.295 43.815))
-    (stroke (width 0) (type default) (color 0 0 0 0))
-  )
   (wire (pts (xy 271.78 144.145) (xy 271.78 146.685))
     (stroke (width 0) (type default) (color 0 0 0 0))
@@
   )
   (wire (pts (xy 265.43 99.06) (xy 265.43 97.79))
-    (stroke (width 0) (type default) (color 0 0 0 0))
-  )
-  (wire (pts (xy 76.835 37.465) (xy 74.295 37.465))
     (stroke (width 0) (type default) (color 0 0 0 0))
   )
@@
     (pin "2")
   )
-  (symbol (lib_id "power:+5V") (at 76.835 37.465 0) (unit 1)
-    (in_bom yes) (on_board yes)
-    (property "Reference" "#PWR0202" (id 0) (at 76.835 41.275 0)
-      (effects (font (size 1.27 1.27)) hide)
-    )
-    (property "Value" "+5V" (id 1) (at 76.835 33.655 0))
-    (property "Footprint" "" (id 2) (at 76.835 37.465 0)
-      (effects (font (size 1.27 1.27)) hide)
-    )
-    (property "Datasheet" "" (id 3) (at 76.835 37.465 0)
+  (symbol (lib_id "power:+5V") (at 90.17 31.75 0) (unit 1)
+    (in_bom yes) (on_board yes)
+    (property "Reference" "#PWR0202" (id 0) (at 90.17 35.56 0)
+      (effects (font (size 1.27 1.27)) hide)
+    )
+    (property "Value" "+5V" (id 1) (at 90.17 27.94 0))
+    (property "Footprint" "" (id 2) (at 90.17 31.75 0)
+      (effects (font (size 1.27 1.27)) hide)
+    )
+    (property "Datasheet" "" (id 3) (at 90.17 31.75 0)
       (effects (font (size 1.27 1.27)) hide)
     )
@@
     (pin "1")
   )
-  (symbol (lib_id "Device:C_Small") (at 79.375 41.275 0) (unit 1)
-    (in_bom yes) (on_board yes)
-    (property "Reference" "C203" (id 0) (at 81.915 40.005 0)
-      (effects (font (size 1.27 1.27)) (justify left))
-    )
-    (property "Value" "100nf" (id 1) (at 81.915 42.545 0)
-      (effects (font (size 1.27 1.27)) (justify left))
-    )
-    (property "Footprint" "Capacitor_SMD:C_0805_2012Metric" (id 2) (at 79.375 41.275 0)
-      (effects (font (size 1.27 1.27)) hide)
-    )
-    (property "Datasheet" "~" (id 3) (at 79.375 41.275 0)
+  (symbol (lib_id "Device:C_Small") (at 90.17 35.56 0) (unit 1)
+    (in_bom yes) (on_board yes)
+    (property "Reference" "C202" (id 0) (at 82.55 34.29 0)
+      (effects (font (size 1.27 1.27)) (justify left))
+    )
+    (property "Value" "100nf" (id 1) (at 82.55 36.83 0)
+      (effects (font (size 1.27 1.27)) (justify left))
+    )
+    (property "Footprint" "Capacitor_SMD:C_0805_2012Metric" (id 2) (at 90.17 35.56 0)
+      (effects (font (size 1.27 1.27)) hide)
+    )
+    (property "Datasheet" "~" (id 3) (at 90.17 35.56 0)
       (effects (font (size 1.27 1.27)) hide)
     )
@@
   (symbol (lib_id "Device:C_Small") (at 141.605 76.835 0) (unit 1)
     (in_bom yes) (on_board yes)
-    (property "Reference" "C205" (id 0) (at 144.145 76.835 0)
+    (property "Reference" "C204" (id 0) (at 144.145 76.835 0)
       (effects (font (size 1.27 1.27)) (justify left))
     )
@@
   (symbol (lib_id "Device:C_Small") (at 132.715 76.835 0) (unit 1)
     (in_bom yes) (on_board yes)
-    (property "Reference" "C204" (id 0) (at 125.095 76.835 0)
+    (property "Reference" "C203" (id 0) (at 125.095 76.835 0)
       (effects (font (size 1.27 1.27)) (justify left))
     )
@@
   (symbol (lib_id "Device:C_Small") (at 75.565 56.515 0) (unit 1)
     (in_bom yes) (on_board yes)
-    (property "Reference" "C202" (id 0) (at 67.945 55.245 0)
+    (property "Reference" "C201" (id 0) (at 67.945 55.245 0)
       (effects (font (size 1.27 1.27)) (justify left))
     )
@@
     (pin "1")
   )
-  (symbol (lib_id "Device:C_Polarized_Small") (at 74.295 41.275 0) (unit 1)
-    (in_bom yes) (on_board yes)
-    (property "Reference" "C201" (id 0) (at 66.675 40.005 0)
-      (effects (font (size 1.27 1.27)) (justify left))
-    )
-    (property "Value" "4.7uf" (id 1) (at 66.675 42.545 0)
-      (effects (font (size 1.27 1.27)) (justify left))
-    )
-    (property "Footprint" "Capacitor_SMD:CP_Elec_4x3" (id 2) (at 74.295 41.275 0)
-      (effects (font (size 1.27 1.27)) hide)
-    )
-    (property "Datasheet" "~" (id 3) (at 74.295 41.275 0)
-      (effects (font (size 1.27 1.27)) hide)
-    )
-    (pin "1")
-    (pin "2")
-  )
   (symbol (lib_id "power:GND") (at 257.175 155.575 0) (unit 1)
     (in_bom yes) (on_board yes)
@@
     (pin "1")
   )
-  (symbol (lib_id "power:GND") (at 76.835 45.085 0) (unit 1)
-    (in_bom yes) (on_board yes)
-    (property "Reference" "#PWR0203" (id 0) (at 76.835 51.435 0)
-      (effects (font (size 1.27 1.27)) hide)
-    )
-    (property "Value" "GND" (id 1) (at 76.835 48.895 0))
-    (property "Footprint" "" (id 2) (at 76.835 45.085 0)
-      (effects (font (size 1.27 1.27)) hide)
-    )
-    (property "Datasheet" "" (id 3) (at 76.835 45.085 0)
-      (effects (font (size 1.27 1.27)) hide)
-    )
+  (symbol (lib_id "power:GND") (at 90.17 39.37 0) (unit 1)
+    (in_bom yes) (on_board yes)
+    (property "Reference" "#PWR0203" (id 0) (at 90.17 45.72 0)
+      (effects (font (size 1.27 1.27)) hide)
+    )
+    (property "Value" "GND" (id 1) (at 90.17 43.18 0))
+    (property "Footprint" "" (id 2) (at 90.17 39.37 0)
+      (effects (font (size 1.27 1.27)) hide)
+    )
+    (property "Datasheet" "" (id 3) (at 90.17 39.37 0)
+      (effects (font (size 1.27 1.27)) hide)
+    )

Commit message: Include fancy ICSP programmer (lol)
Parts:
- added J201: Tag Connect, Connector:Tag-Connect_TC2050-IDC-FP_2x05_P1.27mm_Vertical, symbol Connector_Generic:Conn_02x05_Odd_Even
- added JP201: RSTBridge, Jumper:SolderJumper-2_P1.3mm_Bridged_Pad1.0x1.5mm, symbol Jumper:SolderJumper_2_Bridged
Connections:
- net +5V: now also J201.9 (Pin_9)
- net GND: now also J201.1 (Pin_1)
- net RST: now also JP201.1 (A)
- net ICSP_SCK: now reaches D201.2 (A), U201.17 (PB5)
- net ICSP_SCK: now also J201.4 (Pin_4)
- net ICSP_MOSI: now reaches U201.15 (PB3)
- net ICSP_MOSI: now also J201.10 (Pin_10)
- net ICSP_MISO: now reaches U201.16 (PB4)
- net ICSP_MISO: now also J201.2 (Pin_2)
- new net ICSP_RST: J201.6 (Pin_6), JP201.2 (B)
- no-connect marks 12 -> 14
Other:
- note added: "ICSP"
- moved on the sheet: R201, R202

Commit message: Add breakout for external buttons
Parts:
- added J202: EXT BTN, Connector_JST:JST_EH_S4B-EH_1x04_P2.50mm_Horizontal, symbol Connector:Conn_01x04_Male
Connections:
- net +5V: now also J202.1 (Pin_1)
- net DAY_ADVANCE: now also J202.3 (Pin_3)
- net DAY_RESET: now also J202.4 (Pin_4)
- net DAY_SUBTRACT: now also J202.2 (Pin_2)
Changed lines of the file:
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@@
+    (stroke (width 0) (type default) (color 0 0 0 0))
+  )
+  (wire (pts (xy 210.82 96.52) (xy 191.77 96.52))
     (stroke (width 0) (type default) (color 0 0 0 0))
   )
@@
     (stroke (width 0) (type default) (color 0 0 0 0))
   )
+  (wire (pts (xy 195.58 85.09) (xy 195.58 88.9))
+    (stroke (width 0) (type default) (color 0 0 0 0))
+  )
   (wire (pts (xy 257.175 153.67) (xy 257.175 155.575))
     (stroke (width 0) (type default) (color 0 0 0 0))
@@
     (stroke (width 0) (type default) (color 0 0 0 0))
   )
+  (wire (pts (xy 195.58 88.9) (xy 191.77 88.9))
+    (stroke (width 0) (type default) (color 0 0 0 0))
+  )
+  (wire (pts (xy 210.82 93.98) (xy 191.77 93.98))
+    (stroke (width 0) (type default) (color 0 0 0 0))
+  )
   (wire (pts (xy 90.17 31.75) (xy 90.17 33.02))
     (stroke (width 0) (type default) (color 0 0 0 0))
@@
     (stroke (width 0) (type default) (color 0 0 0 0))
   )
+  (wire (pts (xy 210.82 91.44) (xy 191.77 91.44))
+    (stroke (width 0) (type default) (color 0 0 0 0))
+  )
   (polyline (pts (xy 177.165 75.565) (xy 285.115 75.565))
     (stroke (width 0) (type default) (color 0 0 0 0))
@@
     (effects (font (size 1.27 1.27)) (justify left bottom))
   )
+  (label "DAY_ADVANCE" (at 210.82 93.98 180)
+    (effects (font (size 1.27 1.27)) (justify right bottom))
+  )
   (label "DAY_RESET" (at 126.365 99.695 180)
     (effects (font (size 1.27 1.27)) (justify right bottom))
   )
+  (label "DAY_SUBTRACT" (at 210.82 91.44 180)
+    (effects (font (size 1.27 1.27)) (justify right bottom))
+  )
   (label "ICSP_SCK" (at 140.335 64.135 180)
+    (effects (font (size 1.27 1.27)) (justify right bottom))
+  )
+  (label "DAY_RESET" (at 210.82 96.52 180)
     (effects (font (size 1.27 1.27)) (justify right bottom))
   )
@@
   (hierarchical_label "TXD" (shape output) (at 158.75 97.155 0)
     (effects (font (size 1.27 1.27)) (justify left))
+  )
+  (symbol (lib_id "power:+5V") (at 195.58 85.09 0) (unit 1)
+    (in_bom yes) (on_board yes)
+    (property "Reference" "#PWR0107" (id 0) (at 195.58 88.9 0)
+      (effects (font (size 1.27 1.27)) hide)
+    )
+    (property "Value" "+5V" (id 1) (at 195.58 81.28 0))
+    (property "Footprint" "" (id 2) (at 195.58 85.09 0)
+      (effects (font (size 1.27 1.27)) hide)
+    )
+    (property "Datasheet" "" (id 3) (at 195.58 85.09 0)
+      (effects (font (size 1.27 1.27)) hide)
+    )
+    (pin "1")
   )
   (symbol (lib_id "power:+5V") (at 271.78 127.635 0) (unit 1)
@@
   (symbol (lib_id "Device:R_Small") (at 257.175 134.62 0) (unit 1)
     (in_bom yes) (on_board yes)
-    (property "Reference" "R208" (id 0) (at 251.46 133.35 0)
-      (effects (font (size 1.27 1.27)) (justify left))
-    )
-    (property "Value" "10K" (id 1) (at 251.46 135.89 0)
+    (property "Reference" "R208" (id 0) (at 250.19 133.35 0)
+      (effects (font (size 1.27 1.27)) (justify left))
+    )
+    (property "Value" "10K" (id 1) (at 250.19 135.89 0)
       (effects (font (size 1.27 1.27)) (justify left))
     )
@@
   (symbol (lib_id "Device:R_Small") (at 257.175 151.13 0) (unit 1)
     (in_bom yes) (on_board yes)
-    (property "Reference" "R209" (id 0) (at 251.46 149.86 0)
-      (effects (font (size 1.27 1.27)) (justify left))
-    )
-    (property "Value" "10K" (id 1) (at 251.46 152.4 0)
+    (property "Reference" "R209" (id 0) (at 250.19 149.86 0)
+      (effects (font (size 1.27 1.27)) (justify left))
+    )
+    (property "Value" "10K" (id 1) (at 250.19 152.4 0)
       (effects (font (size 1.27 1.27)) (justify left))
     )
@@
   (symbol (lib_id "Device:R_Small") (at 257.175 117.475 0) (unit 1)
     (in_bom yes) (on_board yes)
-    (property "Reference" "R207" (id 0) (at 251.46 116.205 0)
-      (effects (font (size 1.27 1.27)) (justify left))
-    )
-    (property "Value" "10K" (id 1) (at 251.46 118.745 0)
+    (property "Reference" "R207" (id 0) (at 250.19 115.57 0)
+      (effects (font (size 1.27 1.27)) (justify left))
+    )
+    (property "Value" "10K" (id 1) (at 250.19 118.11 0)
       (effects (font (size 1.27 1.27)) (justify left))
     )
@@
     (pin "2")
   )
+  (symbol (lib_id "Connector:Conn_01x04_Male") (at 186.69 91.44 0) (unit 1)
+    (in_bom yes) (on_board yes)
+    (property "Reference" "J202" (id 0) (at 187.96 100.33 0))
+    (property "Value" "EXT BTN" (id 1) (at 187.96 86.36 0))
+    (property "Footprint" "Connector_JST:JST_EH_S4B-EH_1x04_P2.50mm_Horizontal" (id 2) (at 186.69 91.44 0)
+      (effects (font (size 1.27 1.27)) hide)
+    )
+    (property "Datasheet" "~" (id 3) (at 186.69 91.44 0)
+      (effects (font (size 1.27 1.27)) hide)
+    )
+    (pin "1")
+    (pin "2")
+    (pin "3")
+    (pin "4")
+  )
   (symbol (lib_id "Device:Crystal") (at 137.16 72.39 180) (unit 1)

Commit message: Possible rewire
Connections:
- net +5V: now also J201.2 (Pin_2); no longer J201.9 (Pin_9)
- net GND: now also J201.10 (Pin_10); no longer J201.1 (Pin_1)
- net ICSP_MISO: now also J201.9 (Pin_9); no longer J201.2 (Pin_2)
- net ICSP_MOSI: now also J201.1 (Pin_1); no longer J201.10 (Pin_10)
- net ICSP_RST: now also J201.5 (Pin_5); no longer J201.6 (Pin_6)
- net ICSP_SCK: now also J201.7 (Pin_7); no longer J201.4 (Pin_4)
Other:
- moved on the sheet: J201
Changed lines of the file:
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@@
   (no_connect (at 109.855 107.315))
   (no_connect (at 109.855 81.915))
-  (no_connect (at 163.83 182.245))
   (no_connect (at 79.375 59.055))
+  (no_connect (at 163.83 181.61))
+  (no_connect (at 163.83 184.15))
   (no_connect (at 109.855 109.855))
-  (no_connect (at 163.83 179.705))
+  (no_connect (at 163.83 179.07))
   (no_connect (at 109.855 76.835))
   (no_connect (at 109.855 112.395))
   (no_connect (at 109.855 74.295))
-  (no_connect (at 151.13 179.705))
+  (no_connect (at 151.13 179.07))
   (no_connect (at 109.855 79.375))
-  (no_connect (at 163.83 184.785))
   (no_connect (at 79.375 56.515))
   (no_connect (at 243.205 50.8))
@@
     (stroke (width 0) (type default) (color 0 0 0 0))
   )
+  (wire (pts (xy 139.7 176.53) (xy 151.13 176.53))
+    (stroke (width 0) (type default) (color 0 0 0 0))
+  )
   (wire (pts (xy 134.62 88.9) (xy 111.76 88.9))
     (stroke (width 0) (type default) (color 0 0 0 0))
@@
     (stroke (width 0) (type default) (color 0 0 0 0))
   )
-  (wire (pts (xy 138.43 187.325) (xy 151.13 187.325))
-    (stroke (width 0) (type default) (color 0 0 0 0))
-  )
   (wire (pts (xy 205.74 59.69) (xy 205.74 58.42))
     (stroke (width 0) (type default) (color 0 0 0 0))
@@
     (stroke (width 0) (type default) (color 0 0 0 0))
   )
+  (wire (pts (xy 163.83 176.53) (xy 165.735 176.53))
+    (stroke (width 0) (type default) (color 0 0 0 0))
+  )
   (wire (pts (xy 75.565 51.435) (xy 75.565 53.975))
     (stroke (width 0) (type default) (color 0 0 0 0))
@@
     (stroke (width 0) (type default) (color 0 0 0 0))
   )
+  (wire (pts (xy 165.735 176.53) (xy 165.735 175.26))
+    (stroke (width 0) (type default) (color 0 0 0 0))
+  )
   (wire (pts (xy 250.19 88.9) (xy 250.19 90.17))
     (stroke (width 0) (type default) (color 0 0 0 0))
   )
+  (wire (pts (xy 139.7 186.69) (xy 151.13 186.69))
+    (stroke (width 0) (type default) (color 0 0 0 0))
+  )
   (wire (pts (xy 109.855 97.155) (xy 147.32 97.155))
     (stroke (width 0) (type default) (color 0 0 0 0))
@@
     (stroke (width 0) (type default) (color 0 0 0 0))
   )
-  (wire (pts (xy 138.43 182.245) (xy 151.13 182.245))
-    (stroke (width 0) (type default) (color 0 0 0 0))
-  )
-  (wire (pts (xy 165.735 177.165) (xy 163.83 177.165))
-    (stroke (width 0) (type default) (color 0 0 0 0))
-  )
   (wire (pts (xy 257.175 113.03) (xy 259.08 113.03))
     (stroke (width 0) (type default) (color 0 0 0 0))
@@
     (stroke (width 0) (type default) (color 0 0 0 0))
   )
+  (wire (pts (xy 139.7 181.61) (xy 151.13 181.61))
+    (stroke (width 0) (type default) (color 0 0 0 0))
+  )
   (wire (pts (xy 257.175 113.03) (xy 257.175 114.935))
     (stroke (width 0) (type default) (color 0 0 0 0))
@@
     (stroke (width 0) (type default) (color 0 0 0 0))
   )
-  (wire (pts (xy 138.43 184.785) (xy 151.13 184.785))
+  (wire (pts (xy 163.83 186.69) (xy 165.735 186.69))
     (stroke (width 0) (type default) (color 0 0 0 0))
   )
@@
     (stroke (width 0) (type default) (color 0 0 0 0))
   )
-  (wire (pts (xy 165.735 189.23) (xy 165.735 187.325))
-    (stroke (width 0) (type default) (color 0 0 0 0))
-  )
   (polyline (pts (xy 177.165 165.735) (xy 132.08 165.735))
     (stroke (width 0) (type default) (color 0 0 0 0))
@@
     (stroke (width 0) (type default) (color 0 0 0 0))
   )
-  (wire (pts (xy 165.735 187.325) (xy 163.83 187.325))
-    (stroke (width 0) (type default) (color 0 0 0 0))
-  )
   (polyline (pts (xy 177.165 12.065) (xy 177.165 165.735))
     (stroke (width 0) (type default) (color 0 0 0 0))
@@
     (stroke (width 0) (type default) (color 0 0 0 0))
   )
+  (wire (pts (xy 165.735 186.69) (xy 165.735 188.595))
+    (stroke (width 0) (type default) (color 0 0 0 0))
+  )
   (wire (pts (xy 95.885 42.545) (xy 94.615 42.545))
     (stroke (width 0) (type default) (color 0 0 0 0))
@@
     (stroke (width 0) (type default) (color 0 0 0 0))
   )
-  (wire (pts (xy 138.43 177.165) (xy 151.13 177.165))
-    (stroke (width 0) (type default) (color 0 0 0 0))
-  )
   (wire (pts (xy 271.78 144.145) (xy 271.78 146.685))
     (stroke (width 0) (type default) (color 0 0 0 0))
   )
+  (wire (pts (xy 139.7 184.15) (xy 151.13 184.15))
+    (stroke (width 0) (type default) (color 0 0 0 0))
+  )
   (wire (pts (xy 137.16 81.28) (xy 141.605 81.28))
     (stroke (width 0) (type default) (color 0 0 0 0))
@@
     (stroke (width 0) (type default) (color 0 0 0 0))
   )
-  (wire (pts (xy 165.735 175.26) (xy 165.735 177.165))
-    (stroke (width 0) (type default) (color 0 0 0 0))
-  )
   (wire (pts (xy 116.205 56.515) (xy 109.855 56.515))
     (stroke (width 0) (type default) (color 0 0 0 0))
@@
     (effects (font (size 1.27 1.27)) (justify left bottom))
   )
-  (label "ICSP_MOSI" (at 138.43 177.165 0)
+  (label "ICSP_MOSI" (at 139.7 176.53 0)
     (effects (font (size 1.27 1.27)) (justify left bottom))
   )
@@
     (effects (font (size 1.27 1.27)) (justify right bottom))
   )
-  (label "ICSP_MISO" (at 138.43 187.325 0)
+  (label "ICSP_MISO" (at 139.7 186.69 0)
     (effects (font (size 1.27 1.27)) (justify left bottom))
   )
@@
     (effects (font (size 1.27 1.27)) (justify left bottom))
   )
-  (label "ICSP_SCK" (at 138.43 184.785 0)
+  (label "ICSP_SCK" (at 139.7 184.15 0)
     (effects (font (size 1.27 1.27)) (justify left bottom))
   )
@@
     (effects (font (size 1.27 1.27)) (justify left bottom))
   )
-  (label "ICSP_RST" (at 138.43 182.245 0)
+  (label "ICSP_RST" (at 139.7 181.61 0)
     (effects (font (size 1.27 1.27)) (justify left bottom))
   )
@@
     (pin "1")
   )
-  (symbol (lib_id "Connector_Generic:Conn_02x05_Odd_Even") (at 158.75 182.245 180) (unit 1)
-    (in_bom yes) (on_board yes)
-    (property "Reference" "J201" (id 0) (at 157.48 189.865 0))
-    (property "Value" "Tag Connect" (id 1) (at 154.94 173.99 0))
-    (property "Footprint" "Connector:Tag-Connect_TC2050-IDC-FP_2x05_P1.27mm_Vertical" (id 2) (at 158.75 182.245 0)
-      (effects (font (size 1.27 1.27)) hide)
-    )
-    (property "Datasheet" "~" (id 3) (at 158.75 182.245 0)
+  (symbol (lib_id "Connector_Generic:Conn_02x05_Odd_Even") (at 156.21 181.61 0) (unit 1)
+    (in_bom yes) (on_board yes)
+    (property "Reference" "J201" (id 0) (at 157.48 173.99 0))
+    (property "Value" "Tag Connect" (id 1) (at 156.845 189.23 0))
+    (property "Footprint" "Connector:Tag-Connect_TC2050-IDC-FP_2x05_P1.27mm_Vertical" (id 2) (at 156.21 181.61 0)
+      (effects (font (size 1.27 1.27)) hide)
+    )
+    (property "Datasheet" "~" (id 3) (at 156.21 181.61 0)
       (effects (font (size 1.27 1.27)) hide)
     )
@@
     (pin "1")
   )
-  (symbol (lib_id "power:GND") (at 165.735 189.23 0) (unit 1)
-    (in_bom yes) (on_board yes)
-    (property "Reference" "#PWR0209" (id 0) (at 165.735 195.58 0)
-      (effects (font (size 1.27 1.27)) hide)
-    )
-    (property "Value" "GND" (id 1) (at 165.735 193.04 0))
-    (property "Footprint" "" (id 2) (at 165.735 189.23 0)
-      (effects (font (size 1.27 1.27)) hide)
-    )
-    (property "Datasheet" "" (id 3) (at 165.735 189.23 0)
-      (effects (font (size 1.27 1.27)) hide)
-    )
+  (symbol (lib_id "power:GND") (at 165.735 188.595 0) (unit 1)
+    (in_bom yes) (on_board yes)
+    (property "Reference" "#PWR0209" (id 0) (at 165.735 194.945 0)
+      (effects (font (size 1.27 1.27)) hide)
+    )
+    (property "Value" "GND" (id 1) (at 165.735 192.405 0))
+    (property "Footprint" "" (id 2) (at 165.735 188.595 0)
+      (effects (font (size 1.27 1.27)) hide)
+    )
+    (property "Datasheet" "" (id 3) (at 165.735 188.595 0)
+      (effects (font (size 1.27 1.27)) hide)
+    )
