File: Hardware/Segment_Display_Board/buffer.kicad_sch (KiCad schematic)
At the start: 5 parts, among them Q601 MMBT3904, Q602 MMBT3906

Commit message: Place hardware orders
Parts:
- R603: value 250R -> 240R
Changed lines of the file:
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@@
     (in_bom yes) (on_board yes)
     (property "Reference" "R603" (id 0) (at 167.64 100.965 90))
-    (property "Value" "250R" (id 1) (at 168.91 102.87 90))
+    (property "Value" "240R" (id 1) (at 168.91 102.87 90))
     (property "Footprint" "Resistor_SMD:R_0805_2012Metric" (id 2) (at 170.815 99.06 0)
       (effects (font (size 1.27 1.27)) hide)

Commit message: Fixup some stuff
Parts:
- R603: value 240R -> 270R
Changed lines of the file:
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@@
     (in_bom yes) (on_board yes)
     (property "Reference" "R603" (id 0) (at 167.64 100.965 90))
-    (property "Value" "240R" (id 1) (at 168.91 102.87 90))
+    (property "Value" "270R" (id 1) (at 168.91 102.87 90))
     (property "Footprint" "Resistor_SMD:R_0805_2012Metric" (id 2) (at 170.815 99.06 0)
       (effects (font (size 1.27 1.27)) hide)

Commit message: Works enough to do something basic
Parts:
- R603: value 270R -> 680R
Changed lines of the file:
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@@
     (in_bom yes) (on_board yes)
     (property "Reference" "R603" (id 0) (at 167.64 100.965 90))
-    (property "Value" "270R" (id 1) (at 168.91 102.87 90))
+    (property "Value" "680R" (id 1) (at 168.91 102.87 90))
     (property "Footprint" "Resistor_SMD:R_0805_2012Metric" (id 2) (at 170.815 99.06 0)
       (effects (font (size 1.27 1.27)) hide)

Commit message: Create some doomsday clock stuff
Parts:
- R603: value 680R -> TBD
Other:
- note added: "1k : 19ma 680: 27ma"
Changed lines of the file:
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@@
     (stroke (width 0) (type default) (color 0 0 0 0))
+  )
+  (text "1k : 19ma\n680: 27ma" (at 170.815 109.22 0)
+    (effects (font (size 1.27 1.27)) (justify left bottom))
   )
   (hierarchical_label "OUT" (shape output) (at 185.42 99.06 0)
@@
     (in_bom yes) (on_board yes)
     (property "Reference" "R603" (id 0) (at 167.64 100.965 90))
-    (property "Value" "680R" (id 1) (at 168.91 102.87 90))
+    (property "Value" "TBD" (id 1) (at 168.91 102.87 90))
     (property "Footprint" "Resistor_SMD:R_0805_2012Metric" (id 2) (at 170.815 99.06 0)
       (effects (font (size 1.27 1.27)) hide)
